Commit message: Solved a bug on URDF of webots

File: URDF/khr3hv.urdf (robot description, URDF)
Before this commit: robot khr3hv, 23 links, 22 joints
Joints:
- joint LeftCrus: axis 1 0 0 -> 0 1 0
- joint LeftFemur: axis 1 0 0 -> 0 1 0
- joint LeftFemurHead2: axis 1 0 0 -> 0 1 0
- joint RightCrus: axis 1 0 0 -> 0 1 0
- joint RightFemur: axis 1 0 0 -> 0 1 0
