Commit message: Changed some filenames

File: URDF/nao.urdf (robot description, URDF)
Before this commit: robot NaoH25V50, 79 links, 78 joints
Links:
- link Head: geometry collision mesh filename=meshes/nao_description/meshes/V40/HeadPitch.stl scale=0.1 0.1 0.1; visual mesh filename=meshes/nao_description/meshes/V40/HeadPitch.dae scale=0.1 0.1 0.1
- link LAnklePitch: geometry collision mesh filename=meshes/nao_description/meshes/V40/LAnklePitch.stl scale=0.1 0.1 0.1; visual mesh filename=meshes/nao_description/meshes/V40/LAnklePitch.dae scale=0.1 0.1 0.1
- link LBicep: geometry collision mesh filename=meshes/nao_description/meshes/V40/LShoulderRoll.stl scale=0.1 0.1 0.1; visual mesh filename=meshes/nao_description/meshes/V40/LShoulderRoll.dae scale=0.1 0.1 0.1
- link LFinger11_link: geometry collision mesh filename=meshes/nao_description/meshes/V40/LFinger11.stl scale=0.1 0.1 0.1; visual mesh filename=meshes/nao_description/meshes/V40/LFinger11.dae scale=0.1 0.1 0.1
- link LFinger12_link: geometry collision mesh filename=meshes/nao_description/meshes/V40/LFinger12.stl scale=0.1 0.1 0.1; visual mesh filename=meshes/nao_description/meshes/V40/LFinger12.dae scale=0.1 0.1 0.1
- link LFinger13_link: geometry collision mesh filename=meshes/nao_description/meshes/V40/LFinger13.stl scale=0.1 0.1 0.1; visual mesh filename=meshes/nao_description/meshes/V40/LFinger13.dae scale=0.1 0.1 0.1
- link LFinger21_link: geometry collision mesh filename=meshes/nao_description/meshes/V40/LFinger21.stl scale=0.1 0.1 0.1; visual mesh filename=meshes/nao_description/meshes/V40/LFinger21.dae scale=0.1 0.1 0.1
- link LFinger22_link: geometry collision mesh filename=meshes/nao_description/meshes/V40/LFinger22.stl scale=0.1 0.1 0.1; visual mesh filename=meshes/nao_description/meshes/V40/LFinger22.dae scale=0.1 0.1 0.1
- link LFinger23_link: geometry collision mesh filename=meshes/nao_description/meshes/V40/LFinger23.stl scale=0.1 0.1 0.1; visual mesh filename=meshes/nao_description/meshes/V40/LFinger23.dae scale=0.1 0.1 0.1
- link LForeArm: geometry collision mesh filename=meshes/nao_description/meshes/V40/LElbowRoll.stl scale=0.1 0.1 0.1; visual mesh filename=meshes/nao_description/meshes/V40/LElbowRoll.dae scale=0.1 0.1 0.1
- link LHip: geometry collision mesh filename=meshes/nao_description/meshes/V40/LHipRoll.stl scale=0.1 0.1 0.1; visual mesh filename=meshes/nao_description/meshes/V40/LHipRoll.dae scale=0.1 0.1 0.1
- link LPelvis: geometry collision mesh filename=meshes/nao_description/meshes/V40/LHipYawPitch.stl scale=0.1 0.1 0.1; visual mesh filename=meshes/nao_description/meshes/V40/LHipYawPitch.dae scale=0.1 0.1 0.1
- link LShoulder: geometry collision mesh filename=meshes/nao_description/meshes/V40/LShoulderPitch.stl scale=0.1 0.1 0.1; visual mesh filename=meshes/nao_description/meshes/V40/LShoulderPitch.dae scale=0.1 0.1 0.1
- link LThigh: geometry collision mesh filename=meshes/nao_description/meshes/V40/LHipPitch.stl scale=0.1 0.1 0.1; visual mesh filename=meshes/nao_description/meshes/V40/LHipPitch.dae scale=0.1 0.1 0.1
- link LThumb1_link: geometry collision mesh filename=meshes/nao_description/meshes/V40/LThumb1.stl scale=0.1 0.1 0.1; visual mesh filename=meshes/nao_description/meshes/V40/LThumb1.dae scale=0.1 0.1 0.1
- link LThumb2_link: geometry collision mesh filename=meshes/nao_description/meshes/V40/LThumb2.stl scale=0.1 0.1 0.1; visual mesh filename=meshes/nao_description/meshes/V40/LThumb2.dae scale=0.1 0.1 0.1
- link LTibia: geometry collision mesh filename=meshes/nao_description/meshes/V40/LKneePitch.stl scale=0.1 0.1 0.1; visual mesh filename=meshes/nao_description/meshes/V40/LKneePitch.dae scale=0.1 0.1 0.1
- link Neck: geometry collision mesh filename=meshes/nao_description/meshes/V40/HeadYaw.stl scale=0.1 0.1 0.1; visual mesh filename=meshes/nao_description/meshes/V40/HeadYaw.dae scale=0.1 0.1 0.1
- link RAnklePitch: geometry collision mesh filename=meshes/nao_description/meshes/V40/RAnklePitch.stl scale=0.1 0.1 0.1; visual mesh filename=meshes/nao_description/meshes/V40/RAnklePitch.dae scale=0.1 0.1 0.1
- link RBicep: geometry collision mesh filename=meshes/nao_description/meshes/V40/RShoulderRoll.stl scale=0.1 0.1 0.1; visual mesh filename=meshes/nao_description/meshes/V40/RShoulderRoll.dae scale=0.1 0.1 0.1
- link RFinger11_link: geometry collision mesh filename=meshes/nao_description/meshes/V40/RFinger11.stl scale=0.1 0.1 0.1; visual mesh filename=meshes/nao_description/meshes/V40/RFinger11.dae scale=0.1 0.1 0.1
- link RFinger12_link: geometry collision mesh filename=meshes/nao_description/meshes/V40/RFinger12.stl scale=0.1 0.1 0.1; visual mesh filename=meshes/nao_description/meshes/V40/RFinger12.dae scale=0.1 0.1 0.1
- link RFinger13_link: geometry collision mesh filename=meshes/nao_description/meshes/V40/RFinger13.stl scale=0.1 0.1 0.1; visual mesh filename=meshes/nao_description/meshes/V40/RFinger13.dae scale=0.1 0.1 0.1
- link RFinger21_link: geometry collision mesh filename=meshes/nao_description/meshes/V40/RFinger21.stl scale=0.1 0.1 0.1; visual mesh filename=meshes/nao_description/meshes/V40/RFinger21.dae scale=0.1 0.1 0.1
- link RFinger22_link: geometry collision mesh filename=meshes/nao_description/meshes/V40/RFinger22.stl scale=0.1 0.1 0.1; visual mesh filename=meshes/nao_description/meshes/V40/RFinger22.dae scale=0.1 0.1 0.1
- link RFinger23_link: geometry collision mesh filename=meshes/nao_description/meshes/V40/RFinger23.stl scale=0.1 0.1 0.1; visual mesh filename=meshes/nao_description/meshes/V40/RFinger23.dae scale=0.1 0.1 0.1
- link RForeArm: geometry collision mesh filename=meshes/nao_description/meshes/V40/RElbowRoll.stl scale=0.1 0.1 0.1; visual mesh filename=meshes/nao_description/meshes/V40/RElbowRoll.dae scale=0.1 0.1 0.1
- link RHip: geometry collision mesh filename=meshes/nao_description/meshes/V40/RHipRoll.stl scale=0.1 0.1 0.1; visual mesh filename=meshes/nao_description/meshes/V40/RHipRoll.dae scale=0.1 0.1 0.1
- link RPelvis: geometry collision mesh filename=meshes/nao_description/meshes/V40/RHipYawPitch.stl scale=0.1 0.1 0.1; visual mesh filename=meshes/nao_description/meshes/V40/RHipYawPitch.dae scale=0.1 0.1 0.1
- link RShoulder: geometry collision mesh filename=meshes/nao_description/meshes/V40/RShoulderPitch.stl scale=0.1 0.1 0.1; visual mesh filename=meshes/nao_description/meshes/V40/RShoulderPitch.dae scale=0.1 0.1 0.1
- link RThigh: geometry collision mesh filename=meshes/nao_description/meshes/V40/RHipPitch.stl scale=0.1 0.1 0.1; visual mesh filename=meshes/nao_description/meshes/V40/RHipPitch.dae scale=0.1 0.1 0.1
- link RThumb1_link: geometry collision mesh filename=meshes/nao_description/meshes/V40/RThumb1.stl scale=0.1 0.1 0.1; visual mesh filename=meshes/nao_description/meshes/V40/RThumb1.dae scale=0.1 0.1 0.1
- link RThumb2_link: geometry collision mesh filename=meshes/nao_description/meshes/V40/RThumb2.stl scale=0.1 0.1 0.1; visual mesh filename=meshes/nao_description/meshes/V40/RThumb2.dae scale=0.1 0.1 0.1
- link RTibia: geometry collision mesh filename=meshes/nao_description/meshes/V40/RKneePitch.stl scale=0.1 0.1 0.1; visual mesh filename=meshes/nao_description/meshes/V40/RKneePitch.dae scale=0.1 0.1 0.1
- link l_ankle: geometry collision mesh filename=meshes/nao_description/meshes/V40/LAnkleRoll.stl scale=0.1 0.1 0.1; visual mesh filename=meshes/nao_description/meshes/V40/LAnkleRoll.dae scale=0.1 0.1 0.1
- link l_wrist: geometry collision mesh filename=meshes/nao_description/meshes/V40/LWristYaw.stl scale=0.1 0.1 0.1; visual mesh filename=meshes/nao_description/meshes/V40/LWristYaw.dae scale=0.1 0.1 0.1
- link r_ankle: geometry collision mesh filename=meshes/nao_description/meshes/V40/RAnkleRoll.stl scale=0.1 0.1 0.1; visual mesh filename=meshes/nao_description/meshes/V40/RAnkleRoll.dae scale=0.1 0.1 0.1
- link r_wrist: geometry collision mesh filename=meshes/nao_description/meshes/V40/RWristYaw.stl scale=0.1 0.1 0.1; visual mesh filename=meshes/nao_description/meshes/V40/RWristYaw.dae scale=0.1 0.1 0.1
- link torso: geometry collision mesh filename=meshes/nao_description/meshes/V40/Torso.stl scale=0.1 0.1 0.1; visual mesh filename=meshes/nao_description/meshes/V40/Torso.dae scale=0.1 0.1 0.1
