Commit message: Adjusted visualization for g1, plus solved different bugs

File: URDF/g1.urdf (robot description, URDF)
Before this commit: robot g1_23dof, 33 links, 32 joints
Links:
- link head_link: geometry collision mesh filename=meshes/g1_description/meshes/head_link.dae; visual mesh filename=meshes/g1_description/meshes/head_link.dae
- link left_ankle_pitch_link: geometry collision mesh filename=meshes/g1_description/meshes/left_ankle_pitch_link.dae; visual mesh filename=meshes/g1_description/meshes/left_ankle_pitch_link.dae
- link left_ankle_roll_link: geometry collision sphere radius=0.005; collision sphere radius=0.005
- link left_elbow_link: geometry collision mesh filename=meshes/g1_description/meshes/left_elbow_link.dae; visual mesh filename=meshes/g1_description/meshes/left_elbow_link.dae
- link left_hip_pitch_link: geometry collision mesh filename=meshes/g1_description/meshes/left_hip_pitch_link.dae; visual mesh filename=meshes/g1_description/meshes/left_hip_pitch_link.dae
- link left_hip_roll_link: geometry collision mesh filename=meshes/g1_description/meshes/left_hip_roll_link.dae; visual mesh filename=meshes/g1_description/meshes/left_hip_roll_link.dae
- link left_hip_yaw_link: geometry collision mesh filename=meshes/g1_description/meshes/left_hip_yaw_link.dae; visual mesh filename=meshes/g1_description/meshes/left_hip_yaw_link.dae
- link left_knee_link: geometry collision mesh filename=meshes/g1_description/meshes/left_knee_link.dae; visual mesh filename=meshes/g1_description/meshes/left_knee_link.dae
- link left_shoulder_pitch_link: geometry collision cylinder length=0.05 radius=0.03; visual mesh filename=meshes/g1_description/meshes/left_shoulder_pitch_link.dae
- link left_shoulder_roll_link: geometry collision cylinder length=0.03 radius=0.03; visual mesh filename=meshes/g1_description/meshes/left_shoulder_roll_link.dae
- link left_shoulder_yaw_link: geometry collision mesh filename=meshes/g1_description/meshes/left_shoulder_yaw_link.dae; visual mesh filename=meshes/g1_description/meshes/left_shoulder_yaw_link.dae
- link left_wrist_roll_rubber_hand: geometry collision mesh filename=meshes/g1_description/meshes/left_wrist_roll_rubber_hand.dae; visual mesh filename=meshes/g1_description/meshes/left_wrist_roll_rubber_hand.dae
- link logo_link: geometry collision mesh filename=meshes/g1_description/meshes/logo_link.dae; visual mesh filename=meshes/g1_description/meshes/logo_link.dae
- link pelvis: geometry visual mesh filename=meshes/g1_description/meshes/pelvis.dae
- link pelvis_contour_link: geometry collision mesh filename=meshes/g1_description/meshes/pelvis_contour_link.dae; visual mesh filename=meshes/g1_description/meshes/pelvis_contour_link.dae
- link right_ankle_pitch_link: geometry collision mesh filename=meshes/g1_description/meshes/right_ankle_pitch_link.dae; visual mesh filename=meshes/g1_description/meshes/right_ankle_pitch_link.dae
- link right_ankle_roll_link: geometry collision sphere radius=0.005; collision sphere radius=0.005
- link right_elbow_link: geometry collision mesh filename=meshes/g1_description/meshes/right_elbow_link.dae; visual mesh filename=meshes/g1_description/meshes/right_elbow_link.dae
- link right_hip_pitch_link: geometry collision mesh filename=meshes/g1_description/meshes/right_hip_pitch_link.dae; visual mesh filename=meshes/g1_description/meshes/right_hip_pitch_link.dae
- link right_hip_roll_link: geometry collision mesh filename=meshes/g1_description/meshes/right_hip_roll_link.dae; visual mesh filename=meshes/g1_description/meshes/right_hip_roll_link.dae
- link right_hip_yaw_link: geometry collision mesh filename=meshes/g1_description/meshes/right_hip_yaw_link.dae; visual mesh filename=meshes/g1_description/meshes/right_hip_yaw_link.dae
- link right_knee_link: geometry collision mesh filename=meshes/g1_description/meshes/right_knee_link.dae; visual mesh filename=meshes/g1_description/meshes/right_knee_link.dae
- link right_shoulder_pitch_link: geometry collision cylinder length=0.05 radius=0.03; visual mesh filename=meshes/g1_description/meshes/right_shoulder_pitch_link.dae
- link right_shoulder_roll_link: geometry collision cylinder length=0.03 radius=0.03; visual mesh filename=meshes/g1_description/meshes/right_shoulder_roll_link.dae
- link right_shoulder_yaw_link: geometry collision mesh filename=meshes/g1_description/meshes/right_shoulder_yaw_link.dae; visual mesh filename=meshes/g1_description/meshes/right_shoulder_yaw_link.dae
- link right_wrist_roll_rubber_hand: geometry collision mesh filename=meshes/g1_description/meshes/right_wrist_roll_rubber_hand.d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; visual mesh filename=meshes/g1_description/meshes/right_wrist_roll_rubber_hand.d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
- link torso_link: geometry collision mesh filename=meshes/g1_description/meshes/torso_link.dae; visual mesh filename=meshes/g1_description/meshes/torso_link.dae
- link waist_support_link: geometry collision mesh filename=meshes/g1_description/meshes/waist_support_link.dae; visual mesh filename=meshes/g1_description/meshes/waist_support_link.dae
- link waist_yaw_fixed_link: geometry visual mesh filename=meshes/g1_description/meshes/waist_yaw_link.dae
