Commit message: Fixed URDF bugs and added display python file

File: URDF/atlas.urdf (robot description, URDF)
Before this commit: robot /home/rcatalini/Napoli/Atlas.urdf, 57 links, 56 joints
Links:
- link NeckAy: geometry 
Joints:
- joint LLegKny: origin xyz=-0.05 0 -0.374 rpy=0 -0.000001 0 -> xyz=-0.05 0 -0.374 rpy=0 0 0
- joint LLegLhy: origin xyz=0.05 0 -0.05 rpy=0 -0.000001 0 -> xyz=0.05 0 -0.05 rpy=0 0 0
- joint LLegMhx: origin xyz=0 0 0 rpy=0.000005 0 0 -> xyz=0 0 0 rpy=0 0 0
- joint RArmElx: origin xyz=0 -0.121 0.013 rpy=-0.41889 0 0 -> xyz=0 -0.121 0.013 rpy=0 0 0
- joint RArmShx: origin xyz=0 -0.075 0.036 rpy=-0.75758 0 0 -> xyz=0 -0.075 0.036 rpy=1.373484 0 0
- joint RLegKny: origin xyz=-0.05 0 -0.374 rpy=0 0.000001 0 -> xyz=-0.05 0 -0.374 rpy=0 0 0
- joint RLegLhy: origin xyz=0.05 0 -0.05 rpy=0 0.000002 0 -> xyz=0.05 0 -0.05 rpy=0 0 0
- joint RLegMhx: origin xyz=0 0 0 rpy=-0.000004 0 0 -> xyz=0 0 0 rpy=0 0 0

File: URDF/draco3.urdf (robot description, URDF)
Before this commit: robot draco_3, 48 links, 47 joints
Links:
- link l_ankle_fe_link: geometry visual mesh filename=meshes/draco3_description/meshes/l_ankle_fe_link.stl
- link l_ankle_ie_link: geometry collision box size=0.25 0.15 0.0591; visual mesh filename=meshes/draco3_description/meshes/l_ankle_ie_link.stl
- link l_elbow_fe_link: geometry visual mesh filename=meshes/draco3_description/meshes/l_elbow_fe_link.stl
- link l_hip_aa_link: geometry visual mesh filename=meshes/draco3_description/meshes/l_hip_aa_link.stl
- link l_hip_fe_link: geometry visual mesh filename=meshes/draco3_description/meshes/l_hip_fe_link3.obj
- link l_hip_ie_link: geometry visual mesh filename=meshes/draco3_description/meshes/l_hip_ie_link.stl
- link l_knee_adj_link: geometry visual mesh filename=meshes/draco3_description/meshes/l_knee_adj_link.stl
- link l_knee_fe_ld: geometry visual mesh filename=meshes/draco3_description/meshes/l_knee_fe_ld3.obj
- link l_knee_fe_lp: geometry visual mesh filename=meshes/draco3_description/meshes/l_knee_fe_lp.stl
- link l_sake_gripper_link: geometry visual mesh filename=meshes/draco3_description/meshes/l_sake_gripper_mount.stl
- link l_shoulder_aa_link: geometry visual mesh filename=meshes/draco3_description/meshes/l_shoulder_aa_link.stl
- link l_shoulder_fe_link: geometry visual mesh filename=meshes/draco3_description/meshes/l_shoulder_fe_link.stl
- link l_shoulder_ie_link: geometry visual mesh filename=meshes/draco3_description/meshes/l_shoulder_ie_link3.obj
- link l_wrist_ps_link: geometry visual mesh filename=meshes/draco3_description/meshes/l_wrist_ps_link.stl
- link left_ezgripper_finger_L1_1: geometry visual mesh filename=meshes/draco3_description/meshes/ezgripper_gen2/SAKE_Finger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
- link left_ezgripper_finger_L1_2: geometry visual mesh filename=meshes/draco3_description/meshes/ezgripper_gen2/SAKE_Finger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
- link left_ezgripper_finger_L2_1: geometry collision mesh filename=meshes/draco3_description/meshes/ezgripper_gen2/SAKE_Finger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; visual mesh filename=meshes/draco3_description/meshes/ezgripper_gen2/SAKE_Finger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
- link left_ezgripper_finger_L2_2: geometry collision mesh filename=meshes/draco3_description/meshes/ezgripper_gen2/SAKE_Finger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; visual mesh filename=meshes/draco3_description/meshes/ezgripper_gen2/SAKE_Finger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
- link left_ezgripper_palm_link: geometry visual mesh filename=meshes/draco3_description/meshes/ezgripper_gen2/SAKE_Palm_D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
- link neck_pitch_link: geometry visual mesh filename=meshes/draco3_description/meshes/neck_pitch_link3.obj
- link r_ankle_fe_link: geometry visual mesh filename=meshes/draco3_description/meshes/r_ankle_fe_link.stl
- link r_ankle_ie_link: geometry collision box size=0.25 0.15 0.0591; visual mesh filename=meshes/draco3_description/meshes/r_ankle_ie_link.stl
- link r_elbow_fe_link: geometry visual mesh filename=meshes/draco3_description/meshes/r_elbow_fe_link.stl
- link r_hip_aa_link: geometry visual mesh filename=meshes/draco3_description/meshes/r_hip_aa_link.stl
- link r_hip_fe_link: geometry visual mesh filename=meshes/draco3_description/meshes/r_hip_fe_link3.obj
- link r_hip_ie_link: geometry visual mesh filename=meshes/draco3_description/meshes/r_hip_ie_link.stl
- link r_knee_adj_link: geometry visual mesh filename=meshes/draco3_description/meshes/r_knee_adj_link.stl
- link r_knee_fe_ld: geometry visual mesh filename=meshes/draco3_description/meshes/r_knee_fe_ld3.obj
- link r_knee_fe_lp: geometry visual mesh filename=meshes/draco3_description/meshes/r_knee_fe_lp.stl
- link r_sake_gripper_link: geometry visual mesh filename=meshes/draco3_description/meshes/r_sake_gripper_mount.stl
- link r_shoulder_aa_link: geometry visual mesh filename=meshes/draco3_description/meshes/r_shoulder_aa_link.stl
- link r_shoulder_fe_link: geometry visual mesh filename=meshes/draco3_description/meshes/r_shoulder_fe_link.stl
- link r_shoulder_ie_link: geometry visual mesh filename=meshes/draco3_description/meshes/r_shoulder_ie_link3.obj
- link r_wrist_ps_link: geometry visual mesh filename=meshes/draco3_description/meshes/r_wrist_ps_link.stl
- link right_ezgripper_finger_L1_1: geometry visual mesh filename=meshes/draco3_description/meshes/ezgripper_gen2/SAKE_Finger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
- link right_ezgripper_finger_L1_2: geometry visual mesh filename=meshes/draco3_description/meshes/ezgripper_gen2/SAKE_Finger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
- link right_ezgripper_finger_L2_1: geometry collision mesh filename=meshes/draco3_description/meshes/ezgripper_gen2/SAKE_Finger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; visual mesh filename=meshes/draco3_description/meshes/ezgripper_gen2/SAKE_Finger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
- link right_ezgripper_finger_L2_2: geometry collision mesh filename=meshes/draco3_description/meshes/ezgripper_gen2/SAKE_Finger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; visual mesh filename=meshes/draco3_description/meshes/ezgripper_gen2/SAKE_Finger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
- link right_ezgripper_palm_link: geometry visual mesh filename=meshes/draco3_description/meshes/ezgripper_gen2/SAKE_Palm_D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
- link torso_link: geometry visual mesh filename=meshes/draco3_description/meshes/torso_link3.obj

File: URDF/h1_2.urdf (robot description, URDF)
Before this commit: robot h1_2, 58 links, 57 joints
Links:
- link L_hand_base_link: geometry collision mesh filename=meshes/h1_2_description/meshes/L_hand_base_link.STL; visual mesh filename=meshes/h1_2_description/meshes/L_hand_base_link.STL
- link L_index_intermediate: geometry collision mesh filename=meshes/h1_2_description/meshes/link16_L.STL; visual mesh filename=meshes/h1_2_description/meshes/link16_L.STL
- link L_index_proximal: geometry collision mesh filename=meshes/h1_2_description/meshes/link15_L.STL; visual mesh filename=meshes/h1_2_description/meshes/link15_L.STL
- link L_middle_intermediate: geometry collision mesh filename=meshes/h1_2_description/meshes/link18_L.STL; visual mesh filename=meshes/h1_2_description/meshes/link18_L.STL
- link L_middle_proximal: geometry collision mesh filename=meshes/h1_2_description/meshes/link17_L.STL; visual mesh filename=meshes/h1_2_description/meshes/link17_L.STL
- link L_pinky_intermediate: geometry collision mesh filename=meshes/h1_2_description/meshes/link22_L.STL; visual mesh filename=meshes/h1_2_description/meshes/link22_L.STL
- link L_pinky_proximal: geometry collision mesh filename=meshes/h1_2_description/meshes/link21_L.STL; visual mesh filename=meshes/h1_2_description/meshes/link21_L.STL
- link L_ring_intermediate: geometry collision mesh filename=meshes/h1_2_description/meshes/link20_L.STL; visual mesh filename=meshes/h1_2_description/meshes/link20_L.STL
- link L_ring_proximal: geometry collision mesh filename=meshes/h1_2_description/meshes/link19_L.STL; visual mesh filename=meshes/h1_2_description/meshes/link19_L.STL
- link L_thumb_distal: geometry collision mesh filename=meshes/h1_2_description/meshes/link14_L.STL; visual mesh filename=meshes/h1_2_description/meshes/link14_L.STL
- link L_thumb_intermediate: geometry collision mesh filename=meshes/h1_2_description/meshes/link13_L.STL; visual mesh filename=meshes/h1_2_description/meshes/link13_L.STL
- link L_thumb_proximal: geometry collision mesh filename=meshes/h1_2_description/meshes/link12_L.STL; visual mesh filename=meshes/h1_2_description/meshes/link12_L.STL
- link L_thumb_proximal_base: geometry collision mesh filename=meshes/h1_2_description/meshes/link11_L.STL; visual mesh filename=meshes/h1_2_description/meshes/link11_L.STL
- link R_hand_base_link: geometry collision mesh filename=meshes/h1_2_description/meshes/R_hand_base_link.STL; visual mesh filename=meshes/h1_2_description/meshes/R_hand_base_link.STL
- link R_index_intermediate: geometry collision mesh filename=meshes/h1_2_description/meshes/link16_R.STL; visual mesh filename=meshes/h1_2_description/meshes/link16_R.STL
- link R_index_proximal: geometry collision mesh filename=meshes/h1_2_description/meshes/link15_R.STL; visual mesh filename=meshes/h1_2_description/meshes/link15_R.STL
- link R_middle_intermediate: geometry collision mesh filename=meshes/h1_2_description/meshes/link18_R.STL; visual mesh filename=meshes/h1_2_description/meshes/link18_R.STL
- link R_middle_proximal: geometry collision mesh filename=meshes/h1_2_description/meshes/link17_R.STL; visual mesh filename=meshes/h1_2_description/meshes/link17_R.STL
- link R_pinky_intermediate: geometry collision mesh filename=meshes/h1_2_description/meshes/link22_R.STL; visual mesh filename=meshes/h1_2_description/meshes/link22_R.STL
- link R_pinky_proximal: geometry collision mesh filename=meshes/h1_2_description/meshes/link21_R.STL; visual mesh filename=meshes/h1_2_description/meshes/link21_R.STL
- link R_ring_intermediate: geometry collision mesh filename=meshes/h1_2_description/meshes/link20_R.STL; visual mesh filename=meshes/h1_2_description/meshes/link20_R.STL
- link R_ring_proximal: geometry collision mesh filename=meshes/h1_2_description/meshes/link19_R.STL; visual mesh filename=meshes/h1_2_description/meshes/link19_R.STL
- link R_thumb_distal: geometry collision mesh filename=meshes/h1_2_description/meshes/link14_R.STL; visual mesh filename=meshes/h1_2_description/meshes/link14_R.STL
- link R_thumb_intermediate: geometry collision mesh filename=meshes/h1_2_description/meshes/link13_R.STL; visual mesh filename=meshes/h1_2_description/meshes/link13_R.STL
- link R_thumb_proximal: geometry collision mesh filename=meshes/h1_2_description/meshes/link12_R.STL; visual mesh filename=meshes/h1_2_description/meshes/link12_R.STL
- link R_thumb_proximal_base: geometry collision mesh filename=meshes/h1_2_description/meshes/link11_R.STL; visual mesh filename=meshes/h1_2_description/meshes/link11_R.STL
- link left_ankle_pitch_link: geometry collision mesh filename=meshes/h1_2_description/meshes/left_ankle_pitch_link.STL; visual mesh filename=meshes/h1_2_description/meshes/left_ankle_pitch_link.STL
- link left_ankle_roll_link: geometry collision mesh filename=meshes/h1_2_description/meshes/left_ankle_roll_link.STL; visual mesh filename=meshes/h1_2_description/meshes/left_ankle_roll_link.STL
- link left_elbow_link: geometry collision mesh filename=meshes/h1_2_description/meshes/left_elbow_link.STL; visual mesh filename=meshes/h1_2_description/meshes/left_elbow_link.STL
- link left_hip_pitch_link: geometry collision cylinder length=0.2 radius=0.02; visual mesh filename=meshes/h1_2_description/meshes/left_hip_pitch_link.STL
- link left_hip_roll_link: geometry collision cylinder length=0.01 radius=0.02; visual mesh filename=meshes/h1_2_description/meshes/left_hip_roll_link.STL
- link left_hip_yaw_link: geometry collision cylinder length=0.02 radius=0.01; visual mesh filename=meshes/h1_2_description/meshes/left_hip_yaw_link.STL
- link left_knee_link: geometry collision cylinder length=0.2 radius=0.02; visual mesh filename=meshes/h1_2_description/meshes/left_knee_link.STL
- link left_shoulder_pitch_link: geometry collision mesh filename=meshes/h1_2_description/meshes/left_shoulder_pitch_link.STL; visual mesh filename=meshes/h1_2_description/meshes/left_shoulder_pitch_link.STL
- link left_shoulder_roll_link: geometry collision mesh filename=meshes/h1_2_description/meshes/left_shoulder_roll_link.STL; visual mesh filename=meshes/h1_2_description/meshes/left_shoulder_roll_link.STL
- link left_shoulder_yaw_link: geometry collision mesh filename=meshes/h1_2_description/meshes/left_shoulder_yaw_link.STL; visual mesh filename=meshes/h1_2_description/meshes/left_shoulder_yaw_link.STL
- link left_wrist_pitch_link: geometry collision mesh filename=meshes/h1_2_description/meshes/left_wrist_pitch_link.STL; visual mesh filename=meshes/h1_2_description/meshes/left_wrist_pitch_link.STL
- link left_wrist_roll_link: geometry collision mesh filename=meshes/h1_2_description/meshes/left_wrist_roll_link.STL; visual mesh filename=meshes/h1_2_description/meshes/left_wrist_roll_link.STL
- link left_wrist_yaw_link: geometry visual mesh filename=meshes/h1_2_description/meshes/wrist_yaw_link.STL
- link logo_link: geometry visual mesh filename=meshes/h1_2_description/meshes/logo_link.STL
- link pelvis: geometry collision sphere radius=0.05; visual mesh filename=meshes/h1_2_description/meshes/pelvis.STL
- link right_ankle_pitch_link: geometry collision mesh filename=meshes/h1_2_description/meshes/right_ankle_pitch_link.STL; visual mesh filename=meshes/h1_2_description/meshes/right_ankle_pitch_link.STL
- link right_ankle_roll_link: geometry collision mesh filename=meshes/h1_2_description/meshes/right_ankle_roll_link.STL; visual mesh filename=meshes/h1_2_description/meshes/right_ankle_roll_link.STL
- link right_elbow_link: geometry collision mesh filename=meshes/h1_2_description/meshes/right_elbow_link.STL; visual mesh filename=meshes/h1_2_description/meshes/right_elbow_link.STL
- link right_hip_pitch_link: geometry collision cylinder length=0.2 radius=0.02; visual mesh filename=meshes/h1_2_description/meshes/right_hip_pitch_link.STL
- link right_hip_roll_link: geometry collision cylinder length=0.01 radius=0.02; visual mesh filename=meshes/h1_2_description/meshes/right_hip_roll_link.STL
- link right_hip_yaw_link: geometry collision cylinder length=0.02 radius=0.01; visual mesh filename=meshes/h1_2_description/meshes/right_hip_yaw_link.STL
- link right_knee_link: geometry collision cylinder length=0.2 radius=0.02; visual mesh filename=meshes/h1_2_description/meshes/right_knee_link.STL
- link right_shoulder_pitch_link: geometry collision mesh filename=meshes/h1_2_description/meshes/right_shoulder_pitch_link.STL; visual mesh filename=meshes/h1_2_description/meshes/right_shoulder_pitch_link.STL
- link right_shoulder_roll_link: geometry collision mesh filename=meshes/h1_2_description/meshes/right_shoulder_roll_link.STL; visual mesh filename=meshes/h1_2_description/meshes/right_shoulder_roll_link.STL
- link right_shoulder_yaw_link: geometry collision mesh filename=meshes/h1_2_description/meshes/right_shoulder_yaw_link.STL; visual mesh filename=meshes/h1_2_description/meshes/right_shoulder_yaw_link.STL
- link right_wrist_pitch_link: geometry collision mesh filename=meshes/h1_2_description/meshes/right_wrist_pitch_link.STL; visual mesh filename=meshes/h1_2_description/meshes/right_wrist_pitch_link.STL
- link right_wrist_roll_link: geometry collision mesh filename=meshes/h1_2_description/meshes/right_wrist_roll_link.STL; visual mesh filename=meshes/h1_2_description/meshes/right_wrist_roll_link.STL
- link right_wrist_yaw_link: geometry visual mesh filename=meshes/h1_2_description/meshes/wrist_yaw_link.STL
- link torso_link: geometry collision box size=0.08 0.16 0.1; visual mesh filename=meshes/h1_2_description/meshes/torso_link.STL
