Commit message: Added atlas

File: URDF/atlas.urdf (robot description, URDF)
Before this commit: robot /home/rcatalini/TheCompleteRobot/URDF/atlas.urdf, 57 links, 56 joints
Links:
- removed link BackLbz
- removed link LArmUsy
- removed link LClav
- removed link LFarm
- removed link LFoot
- removed link LHand
- removed link LLarm
- removed link LLegUhz
- removed link LLglut
- removed link LLleg
- removed link LScap
- removed link LTalus
- removed link LUarm
- removed link LUglut
- removed link LUleg
- removed link Ltorso
- removed link Mtorso
- removed link NeckAy
- removed link RArmUsy
- removed link RClav
- removed link RFarm
- removed link RFoot
- removed link RHand
- removed link RLarm
- removed link RLegUhz
- removed link RLglut
- removed link RLleg
- removed link RScap
- removed link RTalus
- removed link RUarm
- removed link RUglut
- removed link RUleg
- removed link Utorso
- removed link base_link
- removed link solid
- removed link solid_0
- removed link solid_1
- removed link solid_10
- removed link solid_11
- removed link solid_12
- removed link solid_13
- removed link solid_14
- removed link solid_15
- removed link solid_16
- removed link solid_17
- removed link solid_18
- removed link solid_19
- removed link solid_2
- removed link solid_20
- removed link solid_3
- removed link solid_4
- removed link solid_5
- removed link solid_6
- removed link solid_7
- removed link solid_8
- removed link solid_9
- added link center_bottom_led_frame, mass 1e-5
- added link center_top_led_frame, mass 1e-5
- added link head, mass 1.41984; collision box size=0.0468 0.12 0.1184; collision box size=0.1311 0.12 0.0591
- added link head_hokuyo_frame, mass 1e-5
- added link head_imu_link, mass 1e-5; visual box size=0.01 0.01 0.01
- added link hokuyo_link, mass 0.057654; collision box size=0.08 0.06 0.04238; collision cylinder length=0.047 radius=0.024425
- added link imu_link, mass 0.1; visual box size=0.01 0.01 0.01
- added link l_clav, mass 2.369; collision box size=0.13 0.15 0.05; collision cylinder length=0.1525 radius=0.045
- added link l_farm, mass 0.981; collision box size=0.135 0.1 0.045; collision cylinder length=0.125 radius=0.045
- added link l_foot, mass 1.634; collision box size=0.26 0.124887 0.05; visual mesh filename=meshes/atlas_description/meshes/l_foot.dae scale=1 1 1
- added link l_hand, mass 2.263; collision box size=0.13 0.09 0.07; collision cylinder length=0.05 radius=0.03
- added link l_larm, mass 2.148; collision box size=0.135 0.15 0.06; collision cylinder length=0.125 radius=0.045
- added link l_lglut, mass 0.69; collision cylinder length=0.060306 radius=0.02009687; collision cylinder length=0.12 radius=0.02
- added link l_lleg, mass 4.367; collision cylinder length=0.40 radius=0.07; visual mesh filename=meshes/atlas_description/meshes/l_lleg.dae scale=1.0 1.0 1.0
- added link l_scap, mass 2.707; collision box size=0.15 0.15 0.06; collision cylinder length=0.125 radius=0.045
- added link l_talus, mass 0.1; collision cylinder length=0.010059 radius=0.010348; collision cylinder length=0.029542 radius=0.010181
- added link l_uarm, mass 1.881; collision box size=0.04 0.07 0.13; collision cylinder length=0.125 radius=0.045
- added link l_uglut, mass 0.5166; collision cylinder length=0.078396 radius=0.019096; collision cylinder length=0.080842 radius=0.019841
- added link l_uleg, mass 7.34; collision cylinder length=0.10 radius=0.1; collision cylinder length=0.15 radius=0.07
- added link left_camera_frame, mass 1e-5
- added link left_camera_optical_frame
- added link left_led_frame, mass 1e-5
- added link ltorso, mass 1.92; visual mesh filename=meshes/atlas_description/meshes/ltorso.dae scale=1 1 1
- added link mtorso, mass 0.55; collision cylinder length=0.02 radius=0.015; collision cylinder length=0.02 radius=0.015
- added link r_clav, mass 2.369; collision box size=0.13 0.15 0.05; collision cylinder length=0.1525 radius=0.045
- added link r_farm, mass 0.981; collision box size=0.135 0.1 0.045; collision cylinder length=0.125 radius=0.045
- added link r_foot, mass 1.634; collision box size=0.26 0.124887 0.05; visual mesh filename=meshes/atlas_description/meshes/r_foot.dae scale=1 1 1
- added link r_hand, mass 2.263; collision box size=0.13 0.09 0.07; collision cylinder length=0.05 radius=0.03
- added link r_larm, mass 2.148; collision box size=0.135 0.15 0.06; collision cylinder length=0.125 radius=0.045
- added link r_lglut, mass 0.69; collision cylinder length=0.060306 radius=0.02009687; collision cylinder length=0.12 radius=0.02
- added link r_lleg, mass 4.367; collision cylinder length=0.40 radius=0.07; visual mesh filename=meshes/atlas_description/meshes/r_lleg.dae scale=1.0 1.0 1.0
- added link r_scap, mass 2.707; collision box size=0.15 0.15 0.06; collision cylinder length=0.125 radius=0.045
- added link r_talus, mass 0.1; collision cylinder length=0.010059 radius=0.010348; collision cylinder length=0.029542 radius=0.010181
- added link r_uarm, mass 1.881; collision box size=0.04 0.07 0.13; collision cylinder length=0.125 radius=0.045
- added link r_uglut, mass 0.5166; collision cylinder length=0.078396 radius=0.019096; collision cylinder length=0.080842 radius=0.019841
- added link r_uleg, mass 7.34; collision cylinder length=0.10 radius=0.1; collision cylinder length=0.15 radius=0.07
- added link right_camera_frame, mass 1e-5
- added link right_camera_optical_frame
- added link right_led_frame, mass 1e-5
- added link utorso, mass 18.484; collision box size=0.3188 0.24 0.3162; collision cylinder length=0.22375 radius=0.0363
- link pelvis: mass None -> 14.2529; geometry collision box size=0.1 0.15 0.2; collision cylinder length=0.05 radius=0.16
Joints:
- removed joint BackLbz
- removed joint BackLbz_Ltorso_joint
- removed joint BackMby
- removed joint BackUbx
- removed joint LArmElx
- removed joint LArmEly
- removed joint LArmMwx
- removed joint LArmShx
- removed joint LArmUsy
- removed joint LArmUsy_LClav_joint
- removed joint LArmUwy
- removed joint LLegKny
- removed joint LLegLax
- removed joint LLegLhy
- removed joint LLegMhx
- removed joint LLegUay
- removed joint LLegUhz
- removed joint LLegUhz_LUglut_joint
- removed joint NeckAy
- removed joint RArmElx
- removed joint RArmEly
- removed joint RArmMwx
- removed joint RArmShx
- removed joint RArmUsy
- removed joint RArmUsy_RClav_joint
- removed joint RArmUwy
- removed joint RLegKny
- removed joint RLegLax
- removed joint RLegLhy
- removed joint RLegMhx
- removed joint RLegUay
- removed joint RLegUhz
- removed joint RLegUhz_RUglut_joint
- removed joint base_link_pelvis_joint
- removed joint solid_0_RUleg_joint
- removed joint solid_10_Utorso_joint
- removed joint solid_11_RScap_joint
- removed joint solid_12_RUarm_joint
- removed joint solid_13_RLarm_joint
- removed joint solid_14_RFarm_joint
- removed joint solid_15_RHand_joint
- removed joint solid_16_LScap_joint
- removed joint solid_17_LUarm_joint
- removed joint solid_18_LLarm_joint
- removed joint solid_19_LFarm_joint
- removed joint solid_1_RLleg_joint
- removed joint solid_20_LHand_joint
- removed joint solid_2_RTalus_joint
- removed joint solid_3_RFoot_joint
- removed joint solid_4_LLglut_joint
- removed joint solid_5_LUleg_joint
- removed joint solid_6_LLleg_joint
- removed joint solid_7_LTalus_joint
- removed joint solid_8_LFoot_joint
- removed joint solid_9_Mtorso_joint
- removed joint solid_RLglut_joint
- added joint back_lbz: type revolute, parent pelvis, child ltorso, origin xyz=-0.0125 0 0 rpy=0 -0 0, axis 0 0 1, limit lower=-0.610865 upper=0.610865 effort=124.016 velocity=12
- added joint back_mby: type revolute, parent ltorso, child mtorso, origin xyz=0 0 0.09 rpy=0 -0 0, axis 0 1 0, limit lower=-1.2 upper=1.28 effort=206.843 velocity=12
- added joint back_ubx: type revolute, parent mtorso, child utorso, origin xyz=0 0 0.05 rpy=0 -0 0, axis 1 0 0, limit lower=-0.790809 upper=0.790809 effort=94.91 velocity=12
- added joint center_bottom_led_frame_joint: type fixed, parent head, child center_bottom_led_frame, origin xyz=0.01125 0.0 -0.0155
- added joint center_top_led_frame_joint: type fixed, parent head, child center_top_led_frame, origin xyz=0.01125 0.0 0.0105
- added joint head_hokuyo_joint: type fixed, parent hokuyo_link, child head_hokuyo_frame, origin xyz=0.03 0 0.015 rpy=0 0 0, axis 0 1 0
- added joint head_imu_joint: type fixed, parent head, child head_imu_link, origin xyz=-0.0475 0.035 0.0 rpy=0 0 0
- added joint hokuyo_joint: type continuous, parent head, child hokuyo_link, origin xyz=-0.0446 0 0.0880 rpy=0 0 0, axis 1 0 0
- added joint imu_joint: type fixed, parent pelvis, child imu_link, origin xyz=0.05991527603 0 -0.01415 rpy=0 0 0
- added joint l_arm_elx: type revolute, parent l_uarm, child l_larm, origin xyz=0 0.121 0.013 rpy=0 -0 0, axis 1 0 0, limit lower=0 upper=2.35619 effort=114 velocity=12
- added joint l_arm_ely: type revolute, parent l_scap, child l_uarm, origin xyz=0 0.185 0 rpy=0 -0 0, axis 0 1 0, limit lower=0 upper=3.14159 effort=114 velocity=12
- added joint l_arm_mwx: type revolute, parent l_farm, child l_hand, origin xyz=0 0.058 0 rpy=0 -0 0, axis 1 0 0, limit lower=-0.436 upper=1.571 effort=60 velocity=12
- added joint l_arm_shx: type revolute, parent l_clav, child l_scap, origin xyz=0 0.075 0.036 rpy=0 -0 0, axis 1 0 0, limit lower=-1.39626 upper=1.74533 effort=170 velocity=12
- added joint l_arm_usy: type revolute, parent utorso, child l_clav, origin xyz=0.024 0.221 0.289 rpy=0 -0 0, axis 0 0.5 0.866025, limit lower=-1.9635 upper=1.9635 effort=212 velocity=12
- added joint l_arm_uwy: type revolute, parent l_larm, child l_farm, origin xyz=0 0.188 -0.013 rpy=0 -0 0, axis 0 1 0, limit lower=-1.571 upper=1.571 effort=114 velocity=12
- added joint l_leg_kny: type revolute, parent l_uleg, child l_lleg, origin xyz=-0.05 0 -0.374 rpy=0 -0 0, axis 0 1 0, limit lower=0 upper=2.45 effort=400 velocity=12
- added joint l_leg_lax: type revolute, parent l_talus, child l_foot, origin xyz=0 0 0 rpy=0 -0 0, axis 1 0 0, limit lower=-0.436 upper=0.436 effort=90 velocity=12
- added joint l_leg_lhy: type revolute, parent l_lglut, child l_uleg, origin xyz=0.05 0 -0.05 rpy=0 -0 0, axis 0 1 0, limit lower=-1.75 upper=0.524 effort=260 velocity=12
- added joint l_leg_mhx: type revolute, parent l_uglut, child l_lglut, origin xyz=0 0 0 rpy=0 -0 0, axis 1 0 0, limit lower=-0.47 upper=0.495 effort=180 velocity=12
- added joint l_leg_uay: type revolute, parent l_lleg, child l_talus, origin xyz=0 0 -0.422 rpy=0 -0 0, axis 0 1 0, limit lower=-0.9 upper=0.698 effort=220 velocity=12
- added joint l_leg_uhz: type revolute, parent pelvis, child l_uglut, origin xyz=0 0.089 0 rpy=0 -0 0, axis 0 0 1, limit lower=-0.32 upper=1.14 effort=110 velocity=12
- added joint left_camera_frame_joint: type fixed, parent head, child left_camera_frame, origin xyz=0.0 0.035 -0.002
- added joint left_camera_optical_frame_joint: type fixed, parent left_camera_frame, child left_camera_optical_frame, origin xyz=0 0 0 rpy=-1.5708 0.0 -1.5708
- added joint left_led_frame_joint: type fixed, parent head, child left_led_frame, origin xyz=-0.01443 0.07452 0.050346 rpy=0 -0.15 0.53
- added joint neck_ay: type revolute, parent utorso, child head, origin xyz=0.21672 0 0.53796 rpy=0 -0 0, axis 0 1 0, limit lower=-0.610865238 upper=1.13446401 effort=5 velocity=12
- added joint r_arm_elx: type revolute, parent r_uarm, child r_larm, origin xyz=0 -0.121 0.013 rpy=0 -0 0, axis 1 0 0, limit lower=-2.35619 upper=0 effort=114 velocity=12
- added joint r_arm_ely: type revolute, parent r_scap, child r_uarm, origin xyz=0 -0.185 0 rpy=0 -0 0, axis 0 1 0, limit lower=0 upper=3.14159 effort=114 velocity=12
- added joint r_arm_mwx: type revolute, parent r_farm, child r_hand, origin xyz=0 -0.058 0 rpy=0 -0 0, axis 1 0 0, limit lower=-1.571 upper=0.436 effort=60 velocity=12
- added joint r_arm_shx: type revolute, parent r_clav, child r_scap, origin xyz=0 -0.075 0.036 rpy=0 -0 0, axis 1 0 0, limit lower=-1.74533 upper=1.39626 effort=170 velocity=12
- added joint r_arm_usy: type revolute, parent utorso, child r_clav, origin xyz=0.024 -0.221 0.289 rpy=0 -0 0, axis 0 0.5 -0.866025, limit lower=-1.9635 upper=1.9635 effort=212 velocity=12
- added joint r_arm_uwy: type revolute, parent r_larm, child r_farm, origin xyz=0 -0.188 -0.013 rpy=0 -0 0, axis 0 1 0, limit lower=-1.571 upper=1.571 effort=114 velocity=12
- added joint r_leg_kny: type revolute, parent r_uleg, child r_lleg, origin xyz=-0.05 0 -0.374 rpy=0 -0 0, axis 0 1 0, limit lower=0 upper=2.45 effort=400 velocity=12
- added joint r_leg_lax: type revolute, parent r_talus, child r_foot, origin xyz=0 0 0 rpy=0 -0 0, axis 1 0 0, limit lower=-0.436 upper=0.436 effort=90 velocity=12
- added joint r_leg_lhy: type revolute, parent r_lglut, child r_uleg, origin xyz=0.05 0 -0.05 rpy=0 -0 0, axis 0 1 0, limit lower=-1.745 upper=0.524 effort=260 velocity=12
- added joint r_leg_mhx: type revolute, parent r_uglut, child r_lglut, origin xyz=0 0 0 rpy=0 -0 0, axis 1 0 0, limit lower=-0.495 upper=0.47 effort=180 velocity=12
- added joint r_leg_uay: type revolute, parent r_lleg, child r_talus, origin xyz=0 0 -0.422 rpy=0 -0 0, axis 0 1 0, limit lower=-0.9 upper=0.698 effort=220 velocity=12
- added joint r_leg_uhz: type revolute, parent pelvis, child r_uglut, origin xyz=0 -0.089 0 rpy=0 -0 0, axis 0 0 1, limit lower=-1.14 upper=0.32 effort=110 velocity=12
- added joint right_camera_frame_joint: type fixed, parent head, child right_camera_frame, origin xyz=0.0 -0.035 -0.002
- added joint right_camera_optical_frame_joint: type fixed, parent right_camera_frame, child right_camera_optical_frame, origin xyz=0 0 0 rpy=-1.5708 0.0 -1.5708
- added joint right_led_frame_joint: type fixed, parent head, child right_led_frame, origin xyz=-0.01443 -0.07452 0.050346 rpy=0 -0.15 -0.53
