Commit message: Added atlas, yet to integrate in  scripts

File: URDF/atlas.urdf (robot description, URDF)
Before this commit: robot atlas, 41 links, 40 joints
Links:
- removed link center_bottom_led_frame
- removed link center_top_led_frame
- removed link head_hokuyo_frame
- removed link head_imu_link
- removed link hokuyo_link
- removed link imu_link
- removed link l_farm
- removed link left_camera_frame
- removed link left_camera_optical_frame
- removed link left_led_frame
- removed link r_farm
- removed link right_camera_frame
- removed link right_camera_optical_frame
- removed link right_led_frame
- added link l_hand_camera_link
- added link l_hand_camera_optical_frame
- added link l_hand_face
- added link l_hand_force_torque, mass 0.1; visual box size=0.01 0.01 0.01
- added link l_hand_gripper
- added link l_lfarm, mass 2.509; collision box size=0.13 0.09 0.07; collision cylinder length=0.05 radius=0.03
- added link l_ufarm, mass 4.386; collision box size=0.135 0.1 0.045; collision cylinder length=0.125 radius=0.045
- added link left_palm; collision mesh filename=meshes/atlasv5_description/meshes/GRIPPER_OPEN_chull.obj scale=1 1 1; visual mesh filename=meshes/atlasv5_description/meshes/GRIPPER_OPEN_chull.obj scale=1 1 1
- added link r_hand_force_torque, mass 0.1; visual box size=0.01 0.01 0.01
- added link r_lfarm, mass 2.509; collision box size=0.13 0.09 0.07; collision cylinder length=0.05 radius=0.03
- added link r_ufarm, mass 4.386; collision box size=0.135 0.1 0.045; collision cylinder length=0.125 radius=0.045
- added link right_palm; collision mesh filename=meshes/atlasv5_description/meshes/GRIPPER_OPEN_chull.obj scale=1 1 1; visual mesh filename=meshes/atlasv5_description/meshes/GRIPPER_OPEN_chull.obj scale=1 1 1
- link head: geometry collision box size=0.0468 0.12 0.1184; collision box size=0.1311 0.12 0.0591
- link l_clav: mass 2.369 -> 4.466; geometry collision box size=0.1 0.07 0.072; collision cylinder length=0.1525 radius=0.0555
- link l_foot: mass 1.634 -> 2.41; geometry collision box size=0.1 0.08 0.02; collision box size=0.227 0.133887 0.05
- link l_hand: mass 2.263 -> 1.0; geometry collision sphere radius=0.03; visual sphere radius=0.03
- link l_larm: mass 2.148 -> 3.248; geometry collision box size=0.135 0.15 0.06; collision cylinder length=0.125 radius=0.045
- link l_lglut: mass 0.69 -> 0.898; geometry collision box size=0.125 0.05 0.08; collision cylinder length=0.060306 radius=0.02009687
- link l_lleg: mass 4.367 -> 4.515; geometry collision cylinder length=0.40 radius=0.07; visual mesh filename=meshes/atlas_description/meshes_unplugged/l_lleg.dae scale=1 1 1
- link l_scap: mass 2.707 -> 3.899; geometry collision box size=0.02 0.029 0.018; collision box size=0.028 0.090 0.05
- link l_talus: mass 0.1 -> 0.125; geometry collision cylinder length=0.010059 radius=0.010348; collision cylinder length=0.029542 radius=0.010181
- link l_uarm: mass 1.881 -> 4.386; geometry collision box size=0.05 0.07 0.15; collision cylinder length=0.11 radius=0.065
- link l_uglut: mass 0.5166 -> 1.959; geometry collision box size=0.05 0.1 0.1; collision cylinder length=0.080842 radius=0.019841
- link l_uleg: mass 7.34 -> 8.204; geometry collision box size=0.07 0.038 0.14; collision box size=0.07 0.038 0.15
- link ltorso: mass 1.92 -> 2.270; geometry visual mesh filename=meshes/atlas_description/meshes_unplugged/ltorso.dae scale=1 1 1
- link mtorso: mass 0.55 -> 0.799; geometry collision cylinder length=0.15 radius=0.02; visual mesh filename=meshes/atlas_description/meshes_unplugged/mtorso.dae scale=1 1 1
- link pelvis: mass 14.2529 -> 9.509; geometry collision box size=0.1 0.15 0.2; collision cylinder length=0.05 radius=0.16
- link r_clav: mass 2.369 -> 4.466; geometry collision box size=0.1 0.07 0.072; collision cylinder length=0.1525 radius=0.0555
- link r_foot: mass 1.634 -> 2.41; geometry collision box size=0.1 0.08 0.02; collision box size=0.227 0.133887 0.05
- link r_hand: mass 2.263 -> 1.0; geometry collision sphere radius=0.03; visual sphere radius=0.03
- link r_larm: mass 2.148 -> 3.248; geometry collision box size=0.135 0.15 0.06; collision cylinder length=0.125 radius=0.045
- link r_lglut: mass 0.69 -> 0.898; geometry collision box size=0.125 0.05 0.08; collision cylinder length=0.060306 radius=0.02009687
- link r_lleg: mass 4.367 -> 4.515; geometry collision cylinder length=0.40 radius=0.07; visual mesh filename=meshes/atlas_description/meshes_unplugged/r_lleg.dae scale=1 1 1
- link r_scap: mass 2.707 -> 3.899; geometry collision box size=0.02 0.029 0.018; collision box size=0.028 0.090 0.05
- link r_talus: mass 0.1 -> 0.125; geometry collision cylinder length=0.010059 radius=0.010348; collision cylinder length=0.029542 radius=0.010181
- link r_uarm: mass 1.881 -> 4.386; geometry collision box size=0.05 0.07 0.15; collision cylinder length=0.11 radius=0.065
- link r_uglut: mass 0.5166 -> 1.959; geometry collision box size=0.05 0.1 0.1; collision cylinder length=0.080842 radius=0.019841
- link r_uleg: mass 7.34 -> 8.204; geometry collision box size=0.07 0.038 0.14; collision box size=0.07 0.038 0.15
- link utorso: mass 18.484 -> 84.409; geometry collision box size=0.13 0.50 0.10; collision box size=0.2 0.18 0.10
Joints:
- removed joint back_lbz
- removed joint back_mby
- removed joint back_ubx
- removed joint center_bottom_led_frame_joint
- removed joint center_top_led_frame_joint
- removed joint head_hokuyo_joint
- removed joint head_imu_joint
- removed joint hokuyo_joint
- removed joint imu_joint
- removed joint l_arm_mwx
- removed joint l_arm_usy
- removed joint l_arm_uwy
- removed joint l_leg_lax
- removed joint l_leg_lhy
- removed joint l_leg_mhx
- removed joint l_leg_uay
- removed joint l_leg_uhz
- removed joint left_camera_frame_joint
- removed joint left_camera_optical_frame_joint
- removed joint left_led_frame_joint
- removed joint neck_ay
- removed joint r_arm_mwx
- removed joint r_arm_usy
- removed joint r_arm_uwy
- removed joint r_leg_lax
- removed joint r_leg_lhy
- removed joint r_leg_mhx
- removed joint r_leg_uay
- removed joint r_leg_uhz
- removed joint right_camera_frame_joint
- removed joint right_camera_optical_frame_joint
- removed joint right_led_frame_joint
- added joint back_bkx: type revolute, parent mtorso, child utorso, origin xyz=0 0 0.05 rpy=0 -0 0, axis 1 0 0, limit lower=-0.523599 upper=0.523599 effort=300 velocity=12
- added joint back_bky: type revolute, parent ltorso, child mtorso, origin xyz=0 0 0.162 rpy=0 -0 0, axis 0 1 0, limit lower=-0.219388 upper=0.538783 effort=445 velocity=9
- added joint back_bkz: type revolute, parent pelvis, child ltorso, origin xyz=-0.0125 0 0 rpy=0 -0 0, axis 0 0 1, limit lower=-0.663225 upper=0.663225 effort=106 velocity=12
- added joint l_arm_shz: type revolute, parent utorso, child l_clav, origin xyz=0.1406 0.2256 0.4776 rpy=0 0 3.14159265359, axis 0 0 1, limit lower=-1.5708 upper=0.785398 effort=87 velocity=12
- added joint l_arm_wrx: type revolute, parent l_ufarm, child l_lfarm, origin xyz=0 -0.119 0.0092 rpy=0 -0 0, axis 1 0 0, limit lower=-1.1781 upper=1.1781 effort=25 velocity=12
- added joint l_arm_wry: type revolute, parent l_larm, child l_ufarm, origin xyz=0 -0.187 -0.0092 rpy=0 3.14159265359 0, axis -0.0 -1.0 -0.0, limit lower=0 upper=3.14159 effort=25 velocity=12
- added joint l_arm_wry2: type revolute, parent l_lfarm, child l_hand, origin xyz=0 0 0 rpy=0 3.14159265359 0, axis 0 1 0, limit lower=-0.001 upper=0.001 effort=5 velocity=1
- added joint l_hand_camera_joint: type fixed, parent l_hand_force_torque, child l_hand_camera_link, origin xyz=-0.09892  0.01431 0.0 rpy= -1.57079 0  1.5708
- added joint l_hand_camera_optical_frame_joint: type fixed, parent l_hand_camera_link, child l_hand_camera_optical_frame, origin xyz=0 0 0 rpy=-1.57079 0.0 -1.57079
- added joint l_hand_face_joint: type fixed, parent l_hand_force_torque, child l_hand_face, origin xyz=0 0.12 0 rpy=0.0 0.0 0.0
- added joint l_hand_force_torque_joint: type fixed, parent l_hand, child l_hand_force_torque, origin xyz=0 -0.1245 0 rpy=0 0 3.141592
- added joint l_hand_gripper_joint: type fixed, parent l_hand_force_torque, child l_hand_gripper, origin xyz=0 0.18 0 rpy=0.0 0.0 0.0
- added joint l_leg_akx: type revolute, parent l_talus, child l_foot, origin xyz=0 0 0 rpy=0 -0 0, axis 1 0 0, limit lower=-0.8 upper=0.8 effort=45 velocity=12
- added joint l_leg_aky: type revolute, parent l_lleg, child l_talus, origin xyz=0 0 -0.422 rpy=0 -0 0, axis 0 1 0, limit lower=-1 upper=0.7 effort=92 velocity=12
- added joint l_leg_hpx: type revolute, parent l_uglut, child l_lglut, origin xyz=0 0 0 rpy=0 -0 0, axis 1 0 0, limit lower=-0.523599 upper=0.523599 effort=530 velocity=12
- added joint l_leg_hpy: type revolute, parent l_lglut, child l_uleg, origin xyz=0.05 0.0225 -0.066 rpy=0 -0 0, axis 0 1 0, limit lower=-1.61234 upper=0.65764 effort=840 velocity=12
- added joint l_leg_hpz: type revolute, parent pelvis, child l_uglut, origin xyz=0 0.089 0 rpy=0 -0 0, axis 0 0 1, limit lower=-0.174358 upper=0.786794 effort=275 velocity=12
- added joint left_palm_joint: type fixed, parent l_hand_force_torque, child left_palm
- added joint neck_ry: type revolute, parent utorso, child head, origin xyz=0.2546 0 0.6215 rpy=0 -0 0, axis 0 1 0, limit lower=-0.602139 upper=1.14319 effort=5 velocity=6.28
- added joint r_arm_shz: type revolute, parent utorso, child r_clav, origin xyz=0.1406 -0.2256 0.4776 rpy=0 -0 0, axis 0 0 1, limit lower=-0.785398 upper=1.5708 effort=87 velocity=12
- added joint r_arm_wrx: type revolute, parent r_ufarm, child r_lfarm, origin xyz=0 -0.119 0.0092 rpy=0 -0 0, axis 1 0 0, limit lower=-1.1781 upper=1.1781 effort=25 velocity=12
- added joint r_arm_wry: type revolute, parent r_larm, child r_ufarm, origin xyz=0 -0.187 -0.0092 rpy=0 -0 0, axis 0 1 0, limit lower=0 upper=3.14159 effort=25 velocity=12
- added joint r_arm_wry2: type revolute, parent r_lfarm, child r_hand, origin xyz=0 0 0 rpy=0 0 0, axis 0 1 0, limit lower=-0.001 upper=0.001 effort=5 velocity=1
- added joint r_hand_force_torque_joint: type fixed, parent r_hand, child r_hand_force_torque, origin xyz=0 -0.1245 0 rpy=0 0 3.141592
- added joint r_leg_akx: type revolute, parent r_talus, child r_foot, origin xyz=0 0 0 rpy=0 -0 0, axis 1 0 0, limit lower=-0.8 upper=0.8 effort=45 velocity=12
- added joint r_leg_aky: type revolute, parent r_lleg, child r_talus, origin xyz=0 0 -0.422 rpy=0 -0 0, axis 0 1 0, limit lower=-1 upper=0.7 effort=92 velocity=12
- added joint r_leg_hpx: type revolute, parent r_uglut, child r_lglut, origin xyz=0 0 0 rpy=0 -0 0, axis 1 0 0, limit lower=-0.523599 upper=0.523599 effort=530 velocity=12
- added joint r_leg_hpy: type revolute, parent r_lglut, child r_uleg, origin xyz=0.05 -0.0225 -0.066 rpy=0 -0 0, axis 0 1 0, limit lower=-1.61234 upper=0.65764 effort=840 velocity=12
- added joint r_leg_hpz: type revolute, parent pelvis, child r_uglut, origin xyz=0 -0.089 0 rpy=0 -0 0, axis 0 0 1, limit lower=-0.786794 upper=0.174358 effort=275 velocity=12
- added joint right_palm_joint: type fixed, parent r_hand_force_torque, child right_palm
- joint l_arm_elx: axis 1 0 0 -> -1.0 -0.0 -0.0; limit lower=0 upper=2.35619 effort=114 velocity=12 -> lower=0 upper=2.35619 effort=112 velocity=12; origin xyz=0 0.121 0.013 rpy=0 -0 0 -> xyz=0 -0.119 0.0092 rpy=0 -0 0
- joint l_arm_ely: axis 0 1 0 -> -0.0 -1.0 -0.0; limit lower=0 upper=3.14159 effort=114 velocity=12 -> lower=0 upper=3.14159 effort=63 velocity=12; origin xyz=0 0.185 0 rpy=0 -0 0 -> xyz=0 -0.187 -0.016 rpy=0 -0 0
- joint l_arm_shx: axis 1 0 0 -> -1.0 -0.0 -0.0; limit lower=-1.39626 upper=1.74533 effort=170 velocity=12 -> lower=-1.5708 upper=1.5708 effort=99 velocity=12; origin xyz=0 0.075 0.036 rpy=0 -0 0 -> xyz=0 -0.11 -0.245 rpy=0 -0 0
- joint l_leg_kny: limit lower=0 upper=2.45 effort=400 velocity=12 -> lower=0 upper=2.35637 effort=890 velocity=12
- joint r_arm_elx: limit lower=-2.35619 upper=0 effort=114 velocity=12 -> lower=-2.35619 upper=0 effort=112 velocity=12; origin xyz=0 -0.121 0.013 rpy=0 -0 0 -> xyz=0 -0.119 0.0092 rpy=0 -0 0
- joint r_arm_ely: limit lower=0 upper=3.14159 effort=114 velocity=12 -> lower=0 upper=3.14159 effort=63 velocity=12; origin xyz=0 -0.185 0 rpy=0 -0 0 -> xyz=0 -0.187 -0.016 rpy=0 -0 0
- joint r_arm_shx: limit lower=-1.74533 upper=1.39626 effort=170 velocity=12 -> lower=-1.5708 upper=1.5708 effort=99 velocity=12; origin xyz=0 -0.075 0.036 rpy=0 -0 0 -> xyz=0 -0.11 -0.245 rpy=0 -0 0
- joint r_leg_kny: limit lower=0 upper=2.45 effort=400 velocity=12 -> lower=0 upper=2.35637 effort=890 velocity=12

Commit message: Some modifications on atlas URDF

File: URDF/atlas.urdf (robot description, URDF)
Before this commit: robot multisense_sl, 39 links, 38 joints
Links:
- link head: geometry collision box size=0.0468 0.12 0.1184; collision box size=0.1311 0.12 0.0591

Commit message: Fixed atlas and some refactoring

File: URDF/atlas.urdf (robot description, URDF)
Before this commit: robot multisense_sl, 39 links, 38 joints
Links:
- removed link l_hand_camera_link
- removed link l_hand_camera_optical_frame
- removed link l_hand_face
- removed link l_hand_force_torque
- removed link l_hand_gripper
- removed link left_palm
- removed link r_hand_force_torque
- removed link right_palm
Joints:
- removed joint l_hand_camera_joint
- removed joint l_hand_camera_optical_frame_joint
- removed joint l_hand_face_joint
- removed joint l_hand_force_torque_joint
- removed joint l_hand_gripper_joint
- removed joint left_palm_joint
- removed joint r_hand_force_torque_joint
- removed joint right_palm_joint
