Commit message: Added Icub

File: URDF/icub.urdf (robot description, URDF)
Before this commit: robot iCub, 213 links, 212 joints
Links:
- removed link chest_ems_gyro_eb1
- removed link chest_ems_gyro_eb2
- removed link chest_ems_gyro_eb3
- removed link chest_ems_gyro_eb4
- removed link head_imu_0
- removed link l_arm_ft_imu
- removed link l_foot_ft
- removed link l_foot_ft_gyro_3b13
- removed link l_forearm_skin_0
- removed link l_forearm_skin_1
- removed link l_forearm_skin_10
- removed link l_forearm_skin_11
- removed link l_forearm_skin_12
- removed link l_forearm_skin_13
- removed link l_forearm_skin_14
- removed link l_forearm_skin_15
- removed link l_forearm_skin_16
- removed link l_forearm_skin_17
- removed link l_forearm_skin_19
- removed link l_forearm_skin_2
- removed link l_forearm_skin_22
- removed link l_forearm_skin_24
- removed link l_forearm_skin_25
- removed link l_forearm_skin_28
- removed link l_forearm_skin_29
- removed link l_forearm_skin_3
- removed link l_forearm_skin_4
- removed link l_forearm_skin_5
- removed link l_forearm_skin_6
- removed link l_forearm_skin_7
- removed link l_forearm_skin_8
- removed link l_forearm_skin_9
- removed link l_lower_leg_ems_gyro_eb7
- removed link l_sole_skin_0
- removed link l_sole_skin_1
- removed link l_sole_skin_10
- removed link l_sole_skin_11
- removed link l_sole_skin_12
- removed link l_sole_skin_13
- removed link l_sole_skin_14
- removed link l_sole_skin_15
- removed link l_sole_skin_17
- removed link l_sole_skin_18
- removed link l_sole_skin_19
- removed link l_sole_skin_2
- removed link l_sole_skin_20
- removed link l_sole_skin_21
- removed link l_sole_skin_22
- removed link l_sole_skin_24
- removed link l_sole_skin_25
- removed link l_sole_skin_26
- removed link l_sole_skin_27
- removed link l_sole_skin_28
- removed link l_sole_skin_29
- removed link l_sole_skin_3
- removed link l_sole_skin_4
- removed link l_sole_skin_8
- removed link l_sole_skin_9
- removed link l_upper_leg_back_contact
- removed link l_upper_leg_dh_frame
- removed link l_upper_leg_ems_gyro_eb10
- removed link l_upper_leg_ems_gyro_eb6
- removed link l_upper_leg_ft_gyro_3b12
- removed link r_arm_ft_imu
- removed link r_foot_ft
- removed link r_foot_ft_gyro_3b14
- removed link r_forearm_skin_0
- removed link r_forearm_skin_1
- removed link r_forearm_skin_10
- removed link r_forearm_skin_11
- removed link r_forearm_skin_12
- removed link r_forearm_skin_13
- removed link r_forearm_skin_14
- removed link r_forearm_skin_15
- removed link r_forearm_skin_16
- removed link r_forearm_skin_17
- removed link r_forearm_skin_19
- removed link r_forearm_skin_2
- removed link r_forearm_skin_22
- removed link r_forearm_skin_24
- removed link r_forearm_skin_25
- removed link r_forearm_skin_28
- removed link r_forearm_skin_29
- removed link r_forearm_skin_3
- removed link r_forearm_skin_4
- removed link r_forearm_skin_5
- removed link r_forearm_skin_6
- removed link r_forearm_skin_7
- removed link r_forearm_skin_8
- removed link r_forearm_skin_9
- removed link r_lower_leg_ems_gyro_eb9
- removed link r_lower_leg_skin_0
- removed link r_lower_leg_skin_10
- removed link r_lower_leg_skin_11
- removed link r_lower_leg_skin_14
- removed link r_lower_leg_skin_15
- removed link r_lower_leg_skin_16
- removed link r_lower_leg_skin_17
- removed link r_lower_leg_skin_19
- removed link r_lower_leg_skin_20
- removed link r_lower_leg_skin_21
- removed link r_lower_leg_skin_28
- removed link r_lower_leg_skin_29
- removed link r_lower_leg_skin_3
- removed link r_lower_leg_skin_31
- removed link r_lower_leg_skin_32
- removed link r_lower_leg_skin_35
- removed link r_lower_leg_skin_36
- removed link r_lower_leg_skin_37
- removed link r_lower_leg_skin_38
- removed link r_lower_leg_skin_4
- removed link r_lower_leg_skin_41
- removed link r_lower_leg_skin_42
- removed link r_lower_leg_skin_43
- removed link r_lower_leg_skin_46
- removed link r_lower_leg_skin_47
- removed link r_lower_leg_skin_49
- removed link r_lower_leg_skin_5
- removed link r_lower_leg_skin_50
- removed link r_lower_leg_skin_51
- removed link r_lower_leg_skin_52
- removed link r_lower_leg_skin_53
- removed link r_lower_leg_skin_54
- removed link r_lower_leg_skin_55
- removed link r_lower_leg_skin_56
- removed link r_lower_leg_skin_6
- removed link r_lower_leg_skin_60
- removed link r_lower_leg_skin_61
- removed link r_lower_leg_skin_9
- removed link r_sole_skin_0
- removed link r_sole_skin_1
- removed link r_sole_skin_10
- removed link r_sole_skin_11
- removed link r_sole_skin_12
- removed link r_sole_skin_13
- removed link r_sole_skin_14
- removed link r_sole_skin_15
- removed link r_sole_skin_17
- removed link r_sole_skin_18
- removed link r_sole_skin_19
- removed link r_sole_skin_2
- removed link r_sole_skin_20
- removed link r_sole_skin_21
- removed link r_sole_skin_22
- removed link r_sole_skin_24
- removed link r_sole_skin_25
- removed link r_sole_skin_26
- removed link r_sole_skin_27
- removed link r_sole_skin_28
- removed link r_sole_skin_29
- removed link r_sole_skin_3
- removed link r_sole_skin_4
- removed link r_sole_skin_8
- removed link r_sole_skin_9
- removed link r_upper_leg_back_contact
- removed link r_upper_leg_dh_frame
- removed link r_upper_leg_ems_gyro_eb11
- removed link r_upper_leg_ems_gyro_eb8
- removed link r_upper_leg_ft_gyro_3b11
- removed link root_link_ems_gyro_eb5
- added link chest_skin_frame, mass 0
- added link codyco_balancing_world, mass 0
- added link l_gripper, mass 0
- added link l_upper_arm_dh_frame, mass 0
- added link r_gripper, mass 0
- added link r_upper_arm_dh_frame, mass 0
- added link torso, mass 0
- link chest: mass 5.638 -> 4.81; geometry collision mesh filename=meshes/iCub_description/meshes/upmc/collision/icub_simple_c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 scale=1 1 1; visual mesh filename=meshes/iCub_description/meshes/upmc/visual/icub_chest.dae scale=1 1 1
- link head: mass 1.50691 -> 1.33687; geometry collision mesh filename=meshes/iCub_description/meshes/upmc/collision/icub_simple_c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 scale=1 1 1; visual mesh filename=meshes/iCub_description/meshes/upmc/visual/icub_head.dae scale=1 1 1
- link imu_frame: mass None -> 0
- link l_ankle_1: mass 0.6798 -> 0.746; geometry collision mesh filename=meshes/iCub_description/meshes/upmc/collision/icub_simple_c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 scale=1 1 1; visual mesh filename=meshes/iCub_description/meshes/upmc/visual/icub_l_ankle_1.d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 scale=1 1 1
- link l_ankle_2: mass 0.265122 -> 0.2675; geometry 
- link l_elbow_1: mass 0.267903 -> 0.074; geometry 
- link l_foot: mass 0.382968 -> 0.5935; geometry collision mesh filename=meshes/iCub_description/meshes/upmc/collision/icub_simple_c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 scale=1 1 1; visual mesh filename=meshes/iCub_description/meshes/upmc/visual/icub_l_foot.dae scale=1 1 1
- link l_foot_dh_frame: mass None -> 0
- link l_forearm: mass 0.636185 -> 0.525; geometry collision mesh filename=meshes/iCub_description/meshes/upmc/collision/icub_simple_c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 scale=1 1 1; visual mesh filename=meshes/iCub_description/meshes/upmc/visual/icub_l_forearm.d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 scale=1 1 1
- link l_forearm_dh_frame: mass None -> 0
- link l_hand: mass 0.247806 -> 0.213; geometry collision mesh filename=meshes/iCub_description/meshes/upmc/collision/icub_simple_c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 scale=1 1 1; visual mesh filename=meshes/iCub_description/meshes/upmc/visual/icub_l_hand.dae scale=1 1 1
- link l_hand_dh_frame: mass None -> 0
- link l_hip_1: mass 0.919725 -> 0.754; geometry collision mesh filename=meshes/iCub_description/meshes/upmc/collision/icub_simple_c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 scale=1 1 1; visual mesh filename=meshes/iCub_description/meshes/upmc/visual/icub_l_hip_1.dae scale=1 1 1
- link l_hip_2: mass 0.415987 -> 0.526; geometry collision mesh filename=meshes/iCub_description/meshes/upmc/collision/icub_simple_c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 scale=1 1 1; visual mesh filename=meshes/iCub_description/meshes/upmc/visual/icub_l_hip_2.dae scale=1 1 1
- link l_hip_3: mass 0.126212 -> 0; geometry 
- link l_lower_leg: mass 1.4724 -> 1.264; geometry collision mesh filename=meshes/iCub_description/meshes/upmc/collision/icub_simple_c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 scale=1 1 1; visual mesh filename=meshes/iCub_description/meshes/upmc/visual/icub_l_shank.dae scale=1 1 1
- link l_shoulder_1: mass 0.114882 -> 0.189; geometry collision mesh filename=meshes/iCub_description/meshes/upmc/collision/icub_simple_c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 scale=1 1 1; visual mesh filename=meshes/iCub_description/meshes/upmc/visual/icub_l_shoulder_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 scale=1 1 1
- link l_shoulder_2: mass 0.238162 -> 0.179; geometry collision mesh filename=meshes/iCub_description/meshes/upmc/collision/icub_simple_c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 scale=1 1 1; visual mesh filename=meshes/iCub_description/meshes/upmc/visual/icub_l_shoulder_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 scale=1 1 1
- link l_shoulder_3: mass 0.35913 -> 0.156157; geometry 
- link l_sole: mass None -> 0
- link l_upper_arm: mass 0.746799 -> 0.727843; geometry collision mesh filename=meshes/iCub_description/meshes/upmc/collision/icub_simple_c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 scale=1 1 1; visual mesh filename=meshes/iCub_description/meshes/upmc/visual/icub_l_arm.dae scale=1 1 1
- link l_upper_leg: mass 1.8084 -> 2.175; geometry collision mesh filename=meshes/iCub_description/meshes/upmc/collision/icub_simple_c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 scale=1 1 1; visual mesh filename=meshes/iCub_description/meshes/upmc/visual/icub_l_thigh.dae scale=1 1 1
- link l_wrist_1: mass 0.0362152 -> 0; geometry 
- link neck_1: mass 0.125793 -> 0; geometry collision mesh filename=meshes/iCub_description/meshes/upmc/collision/icub_simple_c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 scale=1 1 1; visual mesh filename=meshes/iCub_description/meshes/upmc/visual/icub_neck_1.dae scale=1 1 1
- link neck_2: mass 0.177087 -> 0; geometry collision mesh filename=meshes/iCub_description/meshes/upmc/collision/icub_simple_c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 scale=1 1 1; visual mesh filename=meshes/iCub_description/meshes/upmc/visual/icub_neck_2.dae scale=1 1 1
- link r_ankle_1: mass 0.6803 -> 0.746; geometry collision mesh filename=meshes/iCub_description/meshes/upmc/collision/icub_simple_c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 scale=1 1 1; visual mesh filename=meshes/iCub_description/meshes/upmc/visual/icub_r_ankle_1.d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 scale=1 1 1
- link r_ankle_2: mass 0.265122 -> 0.2675; geometry 
- link r_elbow_1: mass 0.267903 -> 0.074; geometry 
- link r_foot: mass 0.382866 -> 0.5935; geometry collision mesh filename=meshes/iCub_description/meshes/upmc/collision/icub_simple_c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 scale=1 1 1; visual mesh filename=meshes/iCub_description/meshes/upmc/visual/icub_r_foot.dae scale=1 1 1
- link r_foot_dh_frame: mass None -> 0
- link r_forearm: mass 0.6347 -> 0.525; geometry collision mesh filename=meshes/iCub_description/meshes/upmc/collision/icub_simple_c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 scale=1 1 1; visual mesh filename=meshes/iCub_description/meshes/upmc/visual/icub_r_forearm.d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 scale=1 1 1
- link r_forearm_dh_frame: mass None -> 0
- link r_hand: mass 0.248289 -> 0.213; geometry collision mesh filename=meshes/iCub_description/meshes/upmc/collision/icub_simple_c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 scale=1 1 1; visual mesh filename=meshes/iCub_description/meshes/upmc/visual/icub_r_hand.dae scale=1 1 1
- link r_hand_dh_frame: mass None -> 0
- link r_hip_1: mass 0.919978 -> 0.754; geometry collision mesh filename=meshes/iCub_description/meshes/upmc/collision/icub_simple_c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 scale=1 1 1; visual mesh filename=meshes/iCub_description/meshes/upmc/visual/icub_r_hip_1.dae scale=1 1 1
- link r_hip_2: mass 0.413242 -> 0.526; geometry collision mesh filename=meshes/iCub_description/meshes/upmc/collision/icub_simple_c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 scale=1 1 1; visual mesh filename=meshes/iCub_description/meshes/upmc/visual/icub_r_hip_2.dae scale=1 1 1
- link r_hip_3: mass 0.126212 -> 0; geometry 
- link r_lower_leg: mass 1.472 -> 1.264; geometry collision mesh filename=meshes/iCub_description/meshes/upmc/collision/icub_simple_c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 scale=1 1 1; visual mesh filename=meshes/iCub_description/meshes/upmc/visual/icub_r_shank.dae scale=1 1 1
- link r_shoulder_1: mass 0.114862 -> 0.189; geometry collision mesh filename=meshes/iCub_description/meshes/upmc/collision/icub_simple_c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 scale=1 1 1; visual mesh filename=meshes/iCub_description/meshes/upmc/visual/icub_r_shoulder_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 scale=1 1 1
- link r_shoulder_2: mass 0.238162 -> 0.179; geometry collision mesh filename=meshes/iCub_description/meshes/upmc/collision/icub_simple_c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 scale=1 1 1; visual mesh filename=meshes/iCub_description/meshes/upmc/visual/icub_r_shoulder_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 scale=1 1 1
- link r_shoulder_3: mass 0.35913 -> 0.155; geometry 
- link r_sole: mass None -> 0
- link r_upper_arm: mass 0.745104 -> 0.729; geometry collision mesh filename=meshes/iCub_description/meshes/upmc/collision/icub_simple_c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 scale=1 1 1; visual mesh filename=meshes/iCub_description/meshes/upmc/visual/icub_r_arm.dae scale=1 1 1
- link r_upper_leg: mass 1.8035 -> 2.175; geometry collision mesh filename=meshes/iCub_description/meshes/upmc/collision/icub_simple_c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 scale=1 1 1; visual mesh filename=meshes/iCub_description/meshes/upmc/visual/icub_r_thigh.dae scale=1 1 1
- link r_wrist_1: mass 0.0362615 -> 0; geometry 
- link root_link: mass 5.09143 -> 4.72; geometry collision mesh filename=meshes/iCub_description/meshes/upmc/collision/icub_simple_c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 scale=1 1 1; visual mesh filename=meshes/iCub_description/meshes/upmc/visual/icub_root_link.d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 scale=1 1 1
- link torso_1: mass 0.67144 -> 0; geometry collision mesh filename=meshes/iCub_description/meshes/upmc/collision/icub_simple_c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 scale=1 1 1; visual mesh filename=meshes/iCub_description/meshes/upmc/visual/icub_lap_belt_1.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 scale=1 1 1
- link torso_2: mass 0.425685 -> 0; geometry 
Joints:
- removed joint base_link_fixed_joint
- removed joint chest_ems_gyro_eb1_fixed_joint
- removed joint chest_ems_gyro_eb2_fixed_joint
- removed joint chest_ems_gyro_eb3_fixed_joint
- removed joint chest_ems_gyro_eb4_fixed_joint
- removed joint head_imu_0_fixed_joint
- removed joint l_arm_ft_imu_fixed_joint
- removed joint l_foot_ft_fixed_joint
- removed joint l_foot_ft_gyro_3b13_fixed_joint
- removed joint l_forearm_skin_0_fixed_joint
- removed joint l_forearm_skin_10_fixed_joint
- removed joint l_forearm_skin_11_fixed_joint
- removed joint l_forearm_skin_12_fixed_joint
- removed joint l_forearm_skin_13_fixed_joint
- removed joint l_forearm_skin_14_fixed_joint
- removed joint l_forearm_skin_15_fixed_joint
- removed joint l_forearm_skin_16_fixed_joint
- removed joint l_forearm_skin_17_fixed_joint
- removed joint l_forearm_skin_19_fixed_joint
- removed joint l_forearm_skin_1_fixed_joint
- removed joint l_forearm_skin_22_fixed_joint
- removed joint l_forearm_skin_24_fixed_joint
- removed joint l_forearm_skin_25_fixed_joint
- removed joint l_forearm_skin_28_fixed_joint
- removed joint l_forearm_skin_29_fixed_joint
- removed joint l_forearm_skin_2_fixed_joint
- removed joint l_forearm_skin_3_fixed_joint
- removed joint l_forearm_skin_4_fixed_joint
- removed joint l_forearm_skin_5_fixed_joint
- removed joint l_forearm_skin_6_fixed_joint
- removed joint l_forearm_skin_7_fixed_joint
- removed joint l_forearm_skin_8_fixed_joint
- removed joint l_forearm_skin_9_fixed_joint
- removed joint l_lower_leg_ems_gyro_eb7_fixed_joint
- removed joint l_sole_skin_0_fixed_joint
- removed joint l_sole_skin_10_fixed_joint
- removed joint l_sole_skin_11_fixed_joint
- removed joint l_sole_skin_12_fixed_joint
- removed joint l_sole_skin_13_fixed_joint
- removed joint l_sole_skin_14_fixed_joint
- removed joint l_sole_skin_15_fixed_joint
- removed joint l_sole_skin_17_fixed_joint
- removed joint l_sole_skin_18_fixed_joint
- removed joint l_sole_skin_19_fixed_joint
- removed joint l_sole_skin_1_fixed_joint
- removed joint l_sole_skin_20_fixed_joint
- removed joint l_sole_skin_21_fixed_joint
- removed joint l_sole_skin_22_fixed_joint
- removed joint l_sole_skin_24_fixed_joint
- removed joint l_sole_skin_25_fixed_joint
- removed joint l_sole_skin_26_fixed_joint
- removed joint l_sole_skin_27_fixed_joint
- removed joint l_sole_skin_28_fixed_joint
- removed joint l_sole_skin_29_fixed_joint
- removed joint l_sole_skin_2_fixed_joint
- removed joint l_sole_skin_3_fixed_joint
- removed joint l_sole_skin_4_fixed_joint
- removed joint l_sole_skin_8_fixed_joint
- removed joint l_sole_skin_9_fixed_joint
- removed joint l_upper_leg_back_contact_fixed_joint
- removed joint l_upper_leg_dh_frame_fixed_joint
- removed joint l_upper_leg_ems_gyro_eb10_fixed_joint
- removed joint l_upper_leg_ems_gyro_eb6_fixed_joint
- removed joint l_upper_leg_ft_gyro_3b12_fixed_joint
- removed joint r_arm_ft_imu_fixed_joint
- removed joint r_foot_ft_fixed_joint
- removed joint r_foot_ft_gyro_3b14_fixed_joint
- removed joint r_forearm_skin_0_fixed_joint
- removed joint r_forearm_skin_10_fixed_joint
- removed joint r_forearm_skin_11_fixed_joint
- removed joint r_forearm_skin_12_fixed_joint
- removed joint r_forearm_skin_13_fixed_joint
- removed joint r_forearm_skin_14_fixed_joint
- removed joint r_forearm_skin_15_fixed_joint
- removed joint r_forearm_skin_16_fixed_joint
- removed joint r_forearm_skin_17_fixed_joint
- removed joint r_forearm_skin_19_fixed_joint
- removed joint r_forearm_skin_1_fixed_joint
- removed joint r_forearm_skin_22_fixed_joint
- removed joint r_forearm_skin_24_fixed_joint
- removed joint r_forearm_skin_25_fixed_joint
- removed joint r_forearm_skin_28_fixed_joint
- removed joint r_forearm_skin_29_fixed_joint
- removed joint r_forearm_skin_2_fixed_joint
- removed joint r_forearm_skin_3_fixed_joint
- removed joint r_forearm_skin_4_fixed_joint
- removed joint r_forearm_skin_5_fixed_joint
- removed joint r_forearm_skin_6_fixed_joint
- removed joint r_forearm_skin_7_fixed_joint
- removed joint r_forearm_skin_8_fixed_joint
- removed joint r_forearm_skin_9_fixed_joint
- removed joint r_lower_leg_ems_gyro_eb9_fixed_joint
- removed joint r_lower_leg_skin_0_fixed_joint
- removed joint r_lower_leg_skin_10_fixed_joint
- removed joint r_lower_leg_skin_11_fixed_joint
- removed joint r_lower_leg_skin_14_fixed_joint
- removed joint r_lower_leg_skin_15_fixed_joint
- removed joint r_lower_leg_skin_16_fixed_joint
- removed joint r_lower_leg_skin_17_fixed_joint
- removed joint r_lower_leg_skin_19_fixed_joint
- removed joint r_lower_leg_skin_20_fixed_joint
- removed joint r_lower_leg_skin_21_fixed_joint
- removed joint r_lower_leg_skin_28_fixed_joint
- removed joint r_lower_leg_skin_29_fixed_joint
- removed joint r_lower_leg_skin_31_fixed_joint
- removed joint r_lower_leg_skin_32_fixed_joint
- removed joint r_lower_leg_skin_35_fixed_joint
- removed joint r_lower_leg_skin_36_fixed_joint
- removed joint r_lower_leg_skin_37_fixed_joint
- removed joint r_lower_leg_skin_38_fixed_joint
- removed joint r_lower_leg_skin_3_fixed_joint
- removed joint r_lower_leg_skin_41_fixed_joint
- removed joint r_lower_leg_skin_42_fixed_joint
- removed joint r_lower_leg_skin_43_fixed_joint
- removed joint r_lower_leg_skin_46_fixed_joint
- removed joint r_lower_leg_skin_47_fixed_joint
- removed joint r_lower_leg_skin_49_fixed_joint
- removed joint r_lower_leg_skin_4_fixed_joint
- removed joint r_lower_leg_skin_50_fixed_joint
- removed joint r_lower_leg_skin_51_fixed_joint
- removed joint r_lower_leg_skin_52_fixed_joint
- removed joint r_lower_leg_skin_53_fixed_joint
- removed joint r_lower_leg_skin_54_fixed_joint
- removed joint r_lower_leg_skin_55_fixed_joint
- removed joint r_lower_leg_skin_56_fixed_joint
- removed joint r_lower_leg_skin_5_fixed_joint
- removed joint r_lower_leg_skin_60_fixed_joint
- removed joint r_lower_leg_skin_61_fixed_joint
- removed joint r_lower_leg_skin_6_fixed_joint
- removed joint r_lower_leg_skin_9_fixed_joint
- removed joint r_sole_skin_0_fixed_joint
- removed joint r_sole_skin_10_fixed_joint
- removed joint r_sole_skin_11_fixed_joint
- removed joint r_sole_skin_12_fixed_joint
- removed joint r_sole_skin_13_fixed_joint
- removed joint r_sole_skin_14_fixed_joint
- removed joint r_sole_skin_15_fixed_joint
- removed joint r_sole_skin_17_fixed_joint
- removed joint r_sole_skin_18_fixed_joint
- removed joint r_sole_skin_19_fixed_joint
- removed joint r_sole_skin_1_fixed_joint
- removed joint r_sole_skin_20_fixed_joint
- removed joint r_sole_skin_21_fixed_joint
- removed joint r_sole_skin_22_fixed_joint
- removed joint r_sole_skin_24_fixed_joint
- removed joint r_sole_skin_25_fixed_joint
- removed joint r_sole_skin_26_fixed_joint
- removed joint r_sole_skin_27_fixed_joint
- removed joint r_sole_skin_28_fixed_joint
- removed joint r_sole_skin_29_fixed_joint
- removed joint r_sole_skin_2_fixed_joint
- removed joint r_sole_skin_3_fixed_joint
- removed joint r_sole_skin_4_fixed_joint
- removed joint r_sole_skin_8_fixed_joint
- removed joint r_sole_skin_9_fixed_joint
- removed joint r_upper_leg_back_contact_fixed_joint
- removed joint r_upper_leg_dh_frame_fixed_joint
- removed joint r_upper_leg_ems_gyro_eb11_fixed_joint
- removed joint r_upper_leg_ems_gyro_eb8_fixed_joint
- removed joint r_upper_leg_ft_gyro_3b11_fixed_joint
- removed joint root_link_ems_gyro_eb5_fixed_joint
- added joint base_fixed_joint: type fixed, parent base_link, child root_link, origin xyz=0 0 0 rpy=0 -0 3.14159265358979323846, axis 0 0 0
- added joint chest_skin_frame_fixed_joint: type fixed, parent chest, child chest_skin_frame, origin xyz=-0.0055 -0.032 3.36778e-19 rpy=1.5708 -1.22465e-16 -3.14159, axis 0 0 0
- added joint codyco_balancing_world_fixed_joint: type fixed, parent l_foot, child codyco_balancing_world, origin xyz=-0.0353 -7.60894e-35 -0.001 rpy=3.14159 -0 0, axis 0 0 0
- added joint l_gripper_joint: type fixed, parent l_hand, child l_gripper, origin xyz=0.0625 0 -0.016 rpy=0 -0 0, axis 0 0 0
- added joint l_upper_arm_dh_frame_fixed_joint: type fixed, parent l_upper_arm, child l_upper_arm_dh_frame, origin xyz=0 0 0.08428 rpy=-1.5708 0 0, axis 0 0 0
- added joint r_gripper_joint: type fixed, parent r_hand, child r_gripper, origin xyz=0.0625 0 0.016 rpy=0 -0 0, axis 0 0 0
- added joint r_upper_arm_dh_frame_fixed_joint: type fixed, parent r_upper_arm, child r_upper_arm_dh_frame, origin xyz=0 0 0.08428 rpy=1.5708 -0 3.14159, axis 0 0 0
- added joint torso_joint: type fixed, parent chest, child torso, origin xyz=0.00231 0.1933 -1.18362e-17 rpy=0 -0 0, axis 0 0 0
- joint imu_frame_fixed_joint: axis (none) -> 0 0 0; origin xyz=0.009500000190735 0.133444 0.009299999999999996 rpy=-1.5707963267948961 1.570796326794896 0 -> xyz=0.0185 -0.1108 0.0066 rpy=1.5708 -0 0
- joint l_ankle_pitch: axis 2.220446049250313e-16 0.9999999999999998 0.0 -> 0 -1 6.12323e-17; limit lower=-0.6108652381980153 upper=0.6108652381980153 effort=37.0 velocity=7.64 -> lower=-0.733038 upper=0.366519 effort=24 velocity=100; origin xyz=0 0 -0.20049999999999996 rpy=0 0 0 -> xyz=-0.213 0 0 rpy=-1.5708 0 0
- joint l_ankle_roll: axis 0.9999999999999998 0.0 2.220446049250313e-16 -> 1 0 0; limit lower=-0.4363323129985824 upper=0.4363323129985824 effort=37.0 velocity=7.64 -> lower=-0.418879 upper=0.418879 effort=11 velocity=100; origin xyz=0 0 0 rpy=0 0 0 -> xyz=0 0 0 rpy=0 -1.5708 0
- joint l_arm_ft_fixed_joint: origin xyz=0.05093014324520106 0 0.029175829465900395 rpy=0 -1.3089970069677395 3.1415926535897927 -> (none); parent l_shoulder_3 -> l_upper_arm
- joint l_arm_ft_sensor: axis (none) -> 0 0 0; origin xyz=0.05093014324520106 0 0.029175829465900395 rpy=0 -1.3089970069677395 3.1415926535897927 -> xyz=0.015 9.36797e-18 0.068 rpy=0 -0 0
- joint l_elbow: axis 2.220446049250313e-16 -1.0000000000000002 0.0 -> 0 1 6.12323e-17; limit lower=0.2617993877991494 upper=1.8500490071139892 effort=50000 velocity=50000 -> lower=0.0959931 upper=1.85005 effort=20 velocity=100; origin xyz=0 0.03399989999999997 0.07925999999999998 rpy=0 -1.3089970069677395 -3.141592653589793 -> xyz=0 0 0.08428 rpy=-6.12323e-17 0 0
- joint l_foot_dh_frame_fixed_joint: origin xyz=0.0 0 0.004 rpy=0 1.5708 0 -> xyz=-0.0353 0 -0.001 rpy=0 1.5708 -0
- joint l_foot_ft_sensor: axis (none) -> 0 0 0; origin xyz=-0.003500000000000003 0 -0.0605 rpy=3.141592653589793 0 0 -> xyz=0.017 0 0.042 rpy=0 -0 0
- joint l_forearm_dh_frame_fixed_joint: axis (none) -> 0 0 0; origin xyz=0.1028711023733811 7.000000000020878e-06 0.027564221311064674 rpy=2.879793333762637 0 1.5707963267948968 -> xyz=0 0.1373 8.4072e-18 rpy=0 -0 0
- joint l_hand_dh_frame_fixed_joint: axis (none) -> 0 0 0; origin xyz=0.05765429784284365 -0.005556799999999987 0.013693832308330513 rpy=-1.5707963267948963 -0.2617993198271562 0 -> xyz=0.0625 0 -0.016 rpy=0 -0 0
- joint l_hip_pitch: axis -2.220446049250313e-16 -0.9999999999999998 0.0 -> 0 -1 6.12323e-17; limit lower=-0.7853981633974483 upper=2.3387411976724017 effort=55.5 velocity=5.1 -> lower=-0.767945 upper=2.30383 effort=84 velocity=100; origin xyz=0.006451499999999999 -0.026000000000000023 -0.11991299999999999 rpy=0 0 -3.141592653589793 -> xyz=0 -0.0681 -0.1199 rpy=0 1.5708 -3.14159
- joint l_hip_roll: axis 0.9999999999999998 0.0 2.220446049250313e-16 -> 1 0 -6.12323e-17; limit lower=-0.3490658503988659 upper=2.0943951023931953 effort=37.0 velocity=7.64 -> lower=-2.07694 upper=0.296706 effort=84 velocity=100; origin xyz=0 0.044099999999999986 0 rpy=0 0 0 -> xyz=0 0 0 rpy=0 -1.5708 3.14159
- joint l_hip_yaw: axis 0.0 2.220446049250313e-16 0.9999999999999998 -> 0 1 6.12323e-17; limit lower=-1.3962634015954636 upper=1.3962634015954636 effort=37.0 velocity=7.64 -> lower=-1.37881 upper=1.37881 effort=40 velocity=100; origin xyz=0 0 0.014399999999999996 rpy=-3.141592653589793 0 0 -> xyz=0 0 -0.0665 rpy=-1.5708 -6.16298e-33 -6.12323e-17
- joint l_knee: axis -2.220446049250313e-16 -0.9999999999999998 0.0 -> 0 1.22465e-16 -1; limit lower=-2.1642082724729685 upper=0.06981317007977318 effort=37.0 velocity=7.64 -> lower=-2.18166 upper=0.401426 effort=30 velocity=100; origin xyz=0 0 -0.14582499999999995 rpy=0 0 0 -> xyz=0 -0.2236 -1.36916e-17 rpy=3.14159 -1.2326e-32 1.5708
- joint l_leg_ft_fixed_joint: origin xyz=0 0 0 rpy=0 0 0 -> (none)
- joint l_leg_ft_sensor: axis (none) -> 0 0 0; origin xyz=-0.0008301999999999962 7.519999999999749e-05 -0.07429999999999995 rpy=3.141592653589793 0 0 -> xyz=0 0 0.0665 rpy=0 -0 0
- joint l_shoulder_pitch: axis 0.965926 0.0 0.258819 -> 0 -1 5.55112e-17; limit lower=-1.6667894356545847 upper=0.17453292519943295 effort=50000 velocity=50000 -> lower=-1.65806 upper=0.0872665 effort=84 velocity=100; origin xyz=0.12001600019073501 0.09280000000000001 0.007969299999999999 rpy=0 0 0 -> xyz=0.00525 0.1433 -0.11026 rpy=1.309 5.55112e-17 1.5708
- joint l_shoulder_roll: axis -0.258819 2.0285226262510233e-17 0.965926 -> 0 1 6.12323e-17; limit lower=0.0 upper=2.8064894372068823 effort=50000 velocity=50000 -> lower=0 upper=2.80649 effort=84 velocity=100; origin xyz=-0.013671000000000016 0 0.0085204 rpy=0.2705973179159596 0.25268017754236044 -1.5015568855866173 -> xyz=0 0 0 rpy=1.5708 -1.11022e-16 -1.5708
- joint l_shoulder_yaw: axis 0.9659258438815126 2.220446049250313e-16 0.2588189794466167 -> 0 6.12323e-17 1; limit lower=-0.6457718232379019 upper=1.3962634015954636 effort=50000 velocity=50000 -> lower=-0.645772 upper=1.74533 effort=34 velocity=100; origin xyz=0.025314346831209797 1.1163643820477631e-07 -0.0054006165626487995 rpy=-0.2526895461750575 -0.008518618321396994 -0.06703988914196896 -> xyz=4.33681e-19 1.73472e-18 0 rpy=6.12323e-17 -0 1.309
- joint l_sole_fixed_joint: axis (none) -> 0 0 0; origin xyz=0.003500000000000003 0 0.0040000000000000036 rpy=-3.141592653589793 0 0 -> xyz=-0.0353 -7.60894e-35 -0.001 rpy=3.14159 -0 0
- joint l_wrist_pitch: axis 0.2588189794466167 0.0 -0.9659258438815124 -> 0 1 6.12323e-17; limit lower=-1.3962634015954636 upper=0.4363323129985824 effort=50000 velocity=50000 -> lower=-1.13446 upper=0.174533 effort=0.65 velocity=100; origin xyz=0.10342756317919133 7.000000000020878e-06 0.025487480746719426 rpy=0 0 0 -> xyz=0 0.1373 8.4072e-18 rpy=1.5708 1.11022e-16 1.5708
- joint l_wrist_prosup: axis 0.9659258438815126 2.220446049250313e-16 0.2588189794466167 -> 0 1 6.12323e-17; limit lower=-1.0471975511965976 upper=1.0471975511965976 effort=50000 velocity=50000 -> lower=-0.872665 upper=0.872665 effort=0.45 velocity=100; origin xyz=0.03846242990265739 0.03399990000000003 -0.0052231681940338075 rpy=0 0 0 -> xyz=-0.015 0 0 rpy=1.5708 -1.11022e-16 -1.5708
- joint l_wrist_yaw: axis -2.220446049250313e-16 1.0000000000000002 0.0 -> 0 0 1; limit lower=-0.3490658503988659 upper=0.4363323129985824 effort=50000 velocity=50000 -> lower=-0.436332 upper=0.436332 effort=0.65 velocity=100; origin xyz=-0.0006341064996442103 -0.0194999 0.0023665183175097023 rpy=0 0 0 -> xyz=0 0 0 rpy=0 -0 0
- joint neck_pitch: axis -1.0 0.0 0.0 -> 0 1 6.12323e-17; limit lower=-0.6981317007977318 upper=0.3839724354387525 effort=50000 velocity=50000 -> lower=-0.698132 upper=0.523599 effort=20 velocity=100; origin xyz=-0.014299999809265 0.17279699999999998 0.005311800000000002 rpy=0 0 0 -> xyz=0.00231 0.1933 -1.18362e-17 rpy=1.5708 1.11022e-16 1.5708
- joint neck_roll: axis 0.0 0.0 1.0 -> 0 -1 6.12323e-17; limit lower=-0.3490658503988659 upper=0.3490658503988659 effort=50000 velocity=50000 -> lower=-1.22173 upper=1.0472 effort=20 velocity=100; origin xyz=0.014299999809265 0.009500000000000008 0.020799969999999997 rpy=0 0 0 -> xyz=0.0095 0 0 rpy=-1.5708 1.11022e-16 -1.5708
- joint neck_yaw: axis 0.0 1.0 0.0 -> 0 -1 6.12323e-17; limit lower=-0.8726646259971648 upper=0.8726646259971648 effort=50000 velocity=50000 -> lower=-0.959931 upper=0.959931 effort=20 velocity=100; origin xyz=0 -0.022344000000000003 -0.020799969999999997 rpy=0 0 0 -> xyz=-5.77779e-34 0 0 rpy=-1.5708 -1.11022e-16 1.5708
- joint r_ankle_pitch: axis 2.220446049250313e-16 0.9999999999999998 0.0 -> 0 1 6.12323e-17; limit lower=-0.6108652381980153 upper=0.6108652381980153 effort=37.0 velocity=7.64 -> lower=-0.733038 upper=0.366519 effort=24 velocity=100; origin xyz=0 0 -0.20049999999999996 rpy=0 0 0 -> xyz=-0.213 0 0 rpy=1.5708 -0 0
- joint r_ankle_roll: axis -0.9999999999999998 0.0 -2.220446049250313e-16 -> -1 1.22465e-16 0; limit lower=-0.4363323129985824 upper=0.4363323129985824 effort=37.0 velocity=7.64 -> lower=-0.418879 upper=0.418879 effort=11 velocity=100; origin xyz=0 0 0 rpy=0 0 0 -> xyz=0 0 0 rpy=0 1.5708 3.14159
- joint r_arm_ft_fixed_joint: origin xyz=-0.05089730176650909 0 0.029167029620599215 rpy=0 -1.3089970069677397 0 -> (none); parent r_shoulder_3 -> r_upper_arm
- joint r_arm_ft_sensor: axis (none) -> 0 0 0; origin xyz=-0.05089730176650909 0 0.029167029620599215 rpy=0 -1.3089970069677397 0 -> xyz=0.015 -8.93429e-18 0.068 rpy=0 -0 0
- joint r_elbow: axis 2.220446049250313e-16 1.0000000000000002 0.0 -> 0 1 6.12323e-17; limit lower=0.2617993877991494 upper=1.8500490071139892 effort=50000 velocity=50000 -> lower=0.0959931 upper=1.85005 effort=20 velocity=100; origin xyz=0 -0.022499900000000003 0.07925999999999998 rpy=0 1.3089970069677397 0 -> xyz=0 0 0.08428 rpy=3.14159 -0 3.14159
- joint r_foot_dh_frame_fixed_joint: origin xyz=0.0 0 0.004 rpy=0 1.5708 0 -> xyz=-0.0353 0 -0.001 rpy=0 1.5708 -0
- joint r_foot_ft_sensor: axis (none) -> 0 0 0; origin xyz=-0.003500000000000003 0 -0.0605 rpy=3.141592653589793 0 0 -> xyz=0.017 0 0.042 rpy=0 -0 0
- joint r_forearm_dh_frame_fixed_joint: axis (none) -> 0 0 0; origin xyz=-0.1028711023733811 7.000000000020878e-06 0.027564221311064674 rpy=-0.26179931982715643 0 -1.5707963267948968 -> xyz=0 -0.1373 -8.4072e-18 rpy=0 -0 0
- joint r_hand_dh_frame_fixed_joint: axis (none) -> 0 0 0; origin xyz=-0.05765429784284365 -0.005556799999999987 0.013693832308330513 rpy=-1.5707963267948963 -0.2617993198271562 3.141592653589793 -> xyz=0.0625 0 0.016 rpy=0 -0 0
- joint r_hip_pitch: axis -2.220446049250313e-16 -0.9999999999999998 0.0 -> 0 1 6.12323e-17; limit lower=-0.7853981633974483 upper=2.3387411976724017 effort=55.5 velocity=5.1 -> lower=-0.767945 upper=2.30383 effort=84 velocity=100; origin xyz=0.006451499999999992 0.025999999999999968 -0.11991299999999999 rpy=0 0 -3.141592653589793 -> xyz=0 0.0681 -0.1199 rpy=0 1.5708 6.12323e-17
- joint r_hip_roll: axis -0.9999999999999998 0.0 -2.220446049250313e-16 -> -1 0 6.12323e-17; limit lower=-0.3490658503988659 upper=2.0943951023931953 effort=37.0 velocity=7.64 -> lower=-2.07694 upper=0.296706 effort=84 velocity=100; origin xyz=0 -0.04409999999999998 0 rpy=0 0 0 -> xyz=0 0 0 rpy=0 1.5708 -6.12323e-17
- joint r_hip_yaw: axis 0.0 -2.220446049250313e-16 -0.9999999999999998 -> 0 -1 6.12323e-17; limit lower=-1.3962634015954636 upper=1.3962634015954636 effort=37.0 velocity=7.64 -> lower=-1.37881 upper=1.37881 effort=40 velocity=100; origin xyz=0 0 0.014399999999999996 rpy=-3.141592653589793 0 0 -> xyz=0 0 -0.0665 rpy=-1.5708 -6.16298e-33 6.12323e-17
- joint r_knee: axis -2.220446049250313e-16 -0.9999999999999998 0.0 -> 0 1.22465e-16 -1; limit lower=-2.1642082724729685 upper=0.06981317007977318 effort=37.0 velocity=7.64 -> lower=-2.18166 upper=0.401426 effort=30 velocity=100; origin xyz=0 0 -0.14582499999999995 rpy=0 0 0 -> xyz=0 -0.2236 1.36916e-17 rpy=3.14159 -1.2326e-32 1.5708
- joint r_leg_ft_fixed_joint: origin xyz=0 0 0 rpy=0 0 0 -> (none)
- joint r_leg_ft_sensor: axis (none) -> 0 0 0; origin xyz=-0.0009362999999999941 1.3899999999969492e-05 -0.07429999999999995 rpy=3.141592653589793 0 0 -> xyz=0 0 0.0665 rpy=0 -0 0
- joint r_shoulder_pitch: axis -0.965925926173269 0.0 0.25881927552505174 -> 0 1 5.55112e-17; limit lower=-1.6667894356545847 upper=0.17453292519943295 effort=50000 velocity=50000 -> lower=-1.65806 upper=0.0872665 effort=84 velocity=100; origin xyz=-0.12001599980926501 0.09280000000000001 0.007969299999999999 rpy=0 -0.523598883792035 3.141592653589793 -> xyz=0.00525 0.1433 0.11026 rpy=-1.309 -0 1.5708
- joint r_shoulder_roll: axis -0.258819 -2.0285226262510233e-17 -0.965926 -> 0 -1 6.12323e-17; limit lower=0.0 upper=2.8064894372068823 effort=50000 velocity=50000 -> lower=0 upper=2.80649 effort=84 velocity=100; origin xyz=-0.007580465732273667 0 0.014210246363868029 rpy=-0.2705976115829963 -0.252680154648383 -1.5015568003498745 -> xyz=0 0 0 rpy=-1.5708 1.11022e-16 -1.5708
- joint r_shoulder_yaw: axis 0.9659258438815126 -2.220446049250313e-16 -0.2588189794466167 -> 0 6.12323e-17 -1; limit lower=-0.6457718232379019 upper=1.3962634015954636 effort=50000 velocity=50000 -> lower=-0.645772 upper=1.74533 effort=34 velocity=100; origin xyz=-0.025346071323150046 2.3275042730641626e-07 -0.0053876480645656255 rpy=-0.2526895461750575 0.008518618321396994 0.06703988914196896 -> xyz=-4.33681e-19 0 0 rpy=3.14159 -0 1.309
- joint r_sole_fixed_joint: axis (none) -> 0 0 0; origin xyz=0.003500000000000003 0 0.0040000000000000036 rpy=-3.141592653589793 0 0 -> xyz=-0.0353 -1.38778e-17 -0.001 rpy=3.14159 -0 0
- joint r_wrist_pitch: axis 0.2588189794466167 0.0 0.9659258438815124 -> 0 1 6.12323e-17; limit lower=-1.3962634015954636 upper=0.4363323129985824 effort=50000 velocity=50000 -> lower=-1.13446 upper=0.174533 effort=0.65 velocity=100; origin xyz=-0.1035052088730253 7.000000000020878e-06 0.02519770299355497 rpy=0 0 0 -> xyz=0 -0.1373 -8.4072e-18 rpy=1.5708 1.11022e-16 1.5708
- joint r_wrist_prosup: axis 0.9659258438815126 -2.220446049250313e-16 -0.2588189794466167 -> 0 1 6.12323e-17; limit lower=-1.0471975511965976 upper=1.0471975511965976 effort=50000 velocity=50000 -> lower=-0.872665 upper=0.872665 effort=0.45 velocity=100; origin xyz=-0.0384624299026574 0.022499900000000017 -0.0052231681940338075 rpy=0 0 0 -> xyz=0.015 0 0 rpy=1.5708 -1.11022e-16 -1.5708
- joint r_wrist_yaw: axis -2.220446049250313e-16 -1.0000000000000002 0.0 -> 0 0 1; limit lower=-0.3490658503988659 upper=0.4363323129985824 effort=50000 velocity=50000 -> lower=-0.436332 upper=0.436332 effort=0.65 velocity=100; origin xyz=0.0006341064996442103 -0.0194999 0.002366518317509704 rpy=0 0 0 -> xyz=0 0 0 rpy=0 -0 3.14159
- joint torso_pitch: axis 1.0 0.0 0.0 -> 0 1 6.12323e-17; limit lower=-0.3490658503988659 upper=1.2217304763960306 effort=50000 velocity=50000 -> lower=-0.383972 upper=1.46608 effort=36 velocity=100; origin xyz=0 0.027046299999999992 0 rpy=1.5707963267948961 0 -1.5707963267948961 -> xyz=0 0 0 rpy=0 -1.5708 3.14159
- joint torso_roll: axis 0.0 0.0 -1.0 -> 0 1 6.12323e-17; limit lower=-0.5235987755982988 upper=0.5235987755982988 effort=50000 velocity=50000 -> lower=-0.680678 upper=0.680678 effort=80 velocity=100; origin xyz=0.027046299809264998 0.032 -0.05734460000000001 rpy=0 0 0 -> xyz=0.032 -2.67276e-51 0 rpy=1.5708 -1.11022e-16 -1.5708
- joint torso_yaw: axis 0.0 -1.0 0.0 -> 0 -1 6.12323e-17; limit lower=-0.8726646259971648 upper=0.8726646259971648 effort=50000 velocity=50000 -> lower=-1.02974 upper=1.02974 effort=80 velocity=100; origin xyz=0 0.05 0.06284210000000001 rpy=0 0 0 -> xyz=-7.46298e-34 -0.0055 0 rpy=-1.5708 1.11022e-16 -1.5708
