Commit message: Inserted Wheeled robot case

File: URDF/pepper.urdf (robot description, URDF)
Before this commit: robot JulietteY20MP, 83 links, 82 joints
Links:
- link Head: geometry collision mesh filename=meshes/pepper_description/meshes/1.0/HeadPitch.stl scale=0.1 0.1 0.1; visual mesh filename=meshes/pepper_description/meshes/1.0/HeadPitch.dae scale=0.1 0.1 0.1
- link Hip: geometry collision mesh filename=meshes/pepper_description/meshes/1.0/HipRoll.stl scale=0.1 0.1 0.1; visual mesh filename=meshes/pepper_description/meshes/1.0/HipRoll.dae scale=0.1 0.1 0.1
- link LBicep: geometry collision mesh filename=meshes/pepper_description/meshes/1.0/LShoulderRoll.stl scale=0.1 0.1 0.1; visual mesh filename=meshes/pepper_description/meshes/1.0/LShoulderRoll.dae scale=0.1 0.1 0.1
- link LElbow: geometry collision mesh filename=meshes/pepper_description/meshes/1.0/LElbowYaw.stl scale=0.1 0.1 0.1; visual mesh filename=meshes/pepper_description/meshes/1.0/LElbowYaw.dae scale=0.1 0.1 0.1
- link LFinger11_link: geometry collision mesh filename=meshes/pepper_description/meshes/1.0/LFinger11.stl scale=0.1 0.1 0.1; visual mesh filename=meshes/pepper_description/meshes/1.0/LFinger11.dae scale=0.1 0.1 0.1
- link LFinger12_link: geometry collision mesh filename=meshes/pepper_description/meshes/1.0/LFinger12.stl scale=0.1 0.1 0.1; visual mesh filename=meshes/pepper_description/meshes/1.0/LFinger12.dae scale=0.1 0.1 0.1
- link LFinger13_link: geometry collision mesh filename=meshes/pepper_description/meshes/1.0/LFinger13.stl scale=0.1 0.1 0.1; visual mesh filename=meshes/pepper_description/meshes/1.0/LFinger13.dae scale=0.1 0.1 0.1
- link LFinger21_link: geometry collision mesh filename=meshes/pepper_description/meshes/1.0/LFinger21.stl scale=0.1 0.1 0.1; visual mesh filename=meshes/pepper_description/meshes/1.0/LFinger21.dae scale=0.1 0.1 0.1
- link LFinger22_link: geometry collision mesh filename=meshes/pepper_description/meshes/1.0/LFinger22.stl scale=0.1 0.1 0.1; visual mesh filename=meshes/pepper_description/meshes/1.0/LFinger22.dae scale=0.1 0.1 0.1
- link LFinger23_link: geometry collision mesh filename=meshes/pepper_description/meshes/1.0/LFinger23.stl scale=0.1 0.1 0.1; visual mesh filename=meshes/pepper_description/meshes/1.0/LFinger23.dae scale=0.1 0.1 0.1
- link LFinger31_link: geometry collision mesh filename=meshes/pepper_description/meshes/1.0/LFinger31.stl scale=0.1 0.1 0.1; visual mesh filename=meshes/pepper_description/meshes/1.0/LFinger31.dae scale=0.1 0.1 0.1
- link LFinger32_link: geometry collision mesh filename=meshes/pepper_description/meshes/1.0/LFinger32.stl scale=0.1 0.1 0.1; visual mesh filename=meshes/pepper_description/meshes/1.0/LFinger32.dae scale=0.1 0.1 0.1
- link LFinger33_link: geometry collision mesh filename=meshes/pepper_description/meshes/1.0/LFinger33.stl scale=0.1 0.1 0.1; visual mesh filename=meshes/pepper_description/meshes/1.0/LFinger33.dae scale=0.1 0.1 0.1
- link LFinger41_link: geometry collision mesh filename=meshes/pepper_description/meshes/1.0/LFinger41.stl scale=0.1 0.1 0.1; visual mesh filename=meshes/pepper_description/meshes/1.0/LFinger41.dae scale=0.1 0.1 0.1
- link LFinger42_link: geometry collision mesh filename=meshes/pepper_description/meshes/1.0/LFinger42.stl scale=0.1 0.1 0.1; visual mesh filename=meshes/pepper_description/meshes/1.0/LFinger42.dae scale=0.1 0.1 0.1
- link LFinger43_link: geometry collision mesh filename=meshes/pepper_description/meshes/1.0/LFinger43.stl scale=0.1 0.1 0.1; visual mesh filename=meshes/pepper_description/meshes/1.0/LFinger43.dae scale=0.1 0.1 0.1
- link LForeArm: geometry collision mesh filename=meshes/pepper_description/meshes/1.0/LElbowRoll.stl scale=0.1 0.1 0.1; visual mesh filename=meshes/pepper_description/meshes/1.0/LElbowRoll.dae scale=0.1 0.1 0.1
- link LShoulder: geometry collision mesh filename=meshes/pepper_description/meshes/1.0/LShoulderPitch.stl scale=0.1 0.1 0.1; visual mesh filename=meshes/pepper_description/meshes/1.0/LShoulderPitch.dae scale=0.1 0.1 0.1
- link LThumb1_link: geometry collision mesh filename=meshes/pepper_description/meshes/1.0/LThumb1.stl scale=0.1 0.1 0.1; visual mesh filename=meshes/pepper_description/meshes/1.0/LThumb1.dae scale=0.1 0.1 0.1
- link LThumb2_link: geometry collision mesh filename=meshes/pepper_description/meshes/1.0/LThumb2.stl scale=0.1 0.1 0.1; visual mesh filename=meshes/pepper_description/meshes/1.0/LThumb2.dae scale=0.1 0.1 0.1
- link Neck: geometry collision mesh filename=meshes/pepper_description/meshes/1.0/HeadYaw.stl scale=0.1 0.1 0.1; visual mesh filename=meshes/pepper_description/meshes/1.0/HeadYaw.dae scale=0.1 0.1 0.1
- link Pelvis: geometry collision mesh filename=meshes/pepper_description/meshes/1.0/HipPitch.stl scale=0.1 0.1 0.1; visual mesh filename=meshes/pepper_description/meshes/1.0/HipPitch.dae scale=0.1 0.1 0.1
- link RBicep: geometry collision mesh filename=meshes/pepper_description/meshes/1.0/RShoulderRoll.stl scale=0.1 0.1 0.1; visual mesh filename=meshes/pepper_description/meshes/1.0/RShoulderRoll.dae scale=0.1 0.1 0.1
- link RElbow: geometry collision mesh filename=meshes/pepper_description/meshes/1.0/RElbowYaw.stl scale=0.1 0.1 0.1; visual mesh filename=meshes/pepper_description/meshes/1.0/RElbowYaw.dae scale=0.1 0.1 0.1
- link RFinger11_link: geometry collision mesh filename=meshes/pepper_description/meshes/1.0/RFinger11.stl scale=0.1 0.1 0.1; visual mesh filename=meshes/pepper_description/meshes/1.0/RFinger11.dae scale=0.1 0.1 0.1
- link RFinger12_link: geometry collision mesh filename=meshes/pepper_description/meshes/1.0/RFinger12.stl scale=0.1 0.1 0.1; visual mesh filename=meshes/pepper_description/meshes/1.0/RFinger12.dae scale=0.1 0.1 0.1
- link RFinger13_link: geometry collision mesh filename=meshes/pepper_description/meshes/1.0/RFinger13.stl scale=0.1 0.1 0.1; visual mesh filename=meshes/pepper_description/meshes/1.0/RFinger13.dae scale=0.1 0.1 0.1
- link RFinger21_link: geometry collision mesh filename=meshes/pepper_description/meshes/1.0/RFinger21.stl scale=0.1 0.1 0.1; visual mesh filename=meshes/pepper_description/meshes/1.0/RFinger21.dae scale=0.1 0.1 0.1
- link RFinger22_link: geometry collision mesh filename=meshes/pepper_description/meshes/1.0/RFinger22.stl scale=0.1 0.1 0.1; visual mesh filename=meshes/pepper_description/meshes/1.0/RFinger22.dae scale=0.1 0.1 0.1
- link RFinger23_link: geometry collision mesh filename=meshes/pepper_description/meshes/1.0/RFinger23.stl scale=0.1 0.1 0.1; visual mesh filename=meshes/pepper_description/meshes/1.0/RFinger23.dae scale=0.1 0.1 0.1
- link RFinger31_link: geometry collision mesh filename=meshes/pepper_description/meshes/1.0/RFinger31.stl scale=0.1 0.1 0.1; visual mesh filename=meshes/pepper_description/meshes/1.0/RFinger31.dae scale=0.1 0.1 0.1
- link RFinger32_link: geometry collision mesh filename=meshes/pepper_description/meshes/1.0/RFinger32.stl scale=0.1 0.1 0.1; visual mesh filename=meshes/pepper_description/meshes/1.0/RFinger32.dae scale=0.1 0.1 0.1
- link RFinger33_link: geometry collision mesh filename=meshes/pepper_description/meshes/1.0/RFinger33.stl scale=0.1 0.1 0.1; visual mesh filename=meshes/pepper_description/meshes/1.0/RFinger33.dae scale=0.1 0.1 0.1
- link RFinger41_link: geometry collision mesh filename=meshes/pepper_description/meshes/1.0/RFinger41.stl scale=0.1 0.1 0.1; visual mesh filename=meshes/pepper_description/meshes/1.0/RFinger41.dae scale=0.1 0.1 0.1
- link RFinger42_link: geometry collision mesh filename=meshes/pepper_description/meshes/1.0/RFinger42.stl scale=0.1 0.1 0.1; visual mesh filename=meshes/pepper_description/meshes/1.0/RFinger42.dae scale=0.1 0.1 0.1
- link RFinger43_link: geometry collision mesh filename=meshes/pepper_description/meshes/1.0/RFinger43.stl scale=0.1 0.1 0.1; visual mesh filename=meshes/pepper_description/meshes/1.0/RFinger43.dae scale=0.1 0.1 0.1
- link RForeArm: geometry collision mesh filename=meshes/pepper_description/meshes/1.0/RElbowRoll.stl scale=0.1 0.1 0.1; visual mesh filename=meshes/pepper_description/meshes/1.0/RElbowRoll.dae scale=0.1 0.1 0.1
- link RShoulder: geometry collision mesh filename=meshes/pepper_description/meshes/1.0/RShoulderPitch.stl scale=0.1 0.1 0.1; visual mesh filename=meshes/pepper_description/meshes/1.0/RShoulderPitch.dae scale=0.1 0.1 0.1
- link RThumb1_link: geometry collision mesh filename=meshes/pepper_description/meshes/1.0/RThumb1.stl scale=0.1 0.1 0.1; visual mesh filename=meshes/pepper_description/meshes/1.0/RThumb1.dae scale=0.1 0.1 0.1
- link RThumb2_link: geometry collision mesh filename=meshes/pepper_description/meshes/1.0/RThumb2.stl scale=0.1 0.1 0.1; visual mesh filename=meshes/pepper_description/meshes/1.0/RThumb2.dae scale=0.1 0.1 0.1
- link Tibia: geometry collision mesh filename=meshes/pepper_description/meshes/1.0/KneePitch.stl scale=0.1 0.1 0.1; visual mesh filename=meshes/pepper_description/meshes/1.0/KneePitch.dae scale=0.1 0.1 0.1
- link WheelB_link: geometry collision mesh filename=meshes/pepper_description/meshes/1.0/WheelB.stl scale=0.1 0.1 0.1; visual mesh filename=meshes/pepper_description/meshes/1.0/WheelB.dae scale=0.1 0.1 0.1
- link WheelFL_link: geometry collision mesh filename=meshes/pepper_description/meshes/1.0/WheelFL.stl scale=0.1 0.1 0.1; visual mesh filename=meshes/pepper_description/meshes/1.0/WheelFL.dae scale=0.1 0.1 0.1
- link WheelFR_link: geometry collision mesh filename=meshes/pepper_description/meshes/1.0/WheelFR.stl scale=0.1 0.1 0.1; visual mesh filename=meshes/pepper_description/meshes/1.0/WheelFR.dae scale=0.1 0.1 0.1
- link l_wrist: geometry collision mesh filename=meshes/pepper_description/meshes/1.0/LWristYaw.stl scale=0.1 0.1 0.1; visual mesh filename=meshes/pepper_description/meshes/1.0/LWristYaw.dae scale=0.1 0.1 0.1
- link r_wrist: geometry collision mesh filename=meshes/pepper_description/meshes/1.0/RWristYaw.stl scale=0.1 0.1 0.1; visual mesh filename=meshes/pepper_description/meshes/1.0/RWristYaw.dae scale=0.1 0.1 0.1
- link torso: geometry collision mesh filename=meshes/pepper_description/meshes/1.0/Torso.stl scale=0.1 0.1 0.1; visual mesh filename=meshes/pepper_description/meshes/1.0/Torso.dae scale=0.1 0.1 0.1

Commit message: Fixed Pepper texture

File: URDF/pepper.urdf (robot description, URDF)
Before this commit: robot JulietteY20MP, 83 links, 82 joints
Links:
- link Head: geometry collision mesh filename=meshes/pepper_description/meshes/1.0/HeadPitch.stl scale=0.1 0.1 0.1; visual mesh filename=meshes/pepper_description/meshes/1.0/HeadPitch_new.dae scale=0.1 0.1 0.1

Commit message: Fixed Icub camera. Spotted probable bug in IK head orientation

File: URDF/pepper.urdf (robot description, URDF)
Before this commit: robot JulietteY20MP, 83 links, 82 joints
Links:
- link Head: geometry collision mesh filename=meshes/pepper_description/meshes/1.0/HeadPitch.stl scale=0.1 0.1 0.1; visual mesh filename=meshes/pepper_description/meshes/1.0/HeadPitch.dae scale=0.1 0.1 0.1
